File: Prototipo_/Prototipo/_autosave-prototipo.kicad_pcb (KiCad board)
At the start: 2 copper layers, 124 parts, among them J1 Conn_01x02_Socket, J4 Conn_01x12_Pin, Q1 MMBT2222A, Q10 MMBT2222A, Q11 MMBT2907A, Q12 MMBT2222A, Q13 MMBT2222A, Q14 MMBT2907A, Q15 MMBT2222A, Q16 MMBT2222A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

Commit message: pruebo modulos de celdas en el esquematico del pcb
Parts:
- moved VCELL1 564.1 mm to (477.9, 209.0)
- moved VCELL2 475.1 mm to (391.4, 210.0)
- moved TP17 394.1 mm to (434.1, 260.4), turned to 0 degrees
- moved Q3 365.1 mm to (421.3, 396.4), turned to 0 degrees
- moved TP9 364.2 mm to (447.9, 455.2), turned to 0 degrees
- moved Q1 359.5 mm to (421.3, 392.0), turned to 0 degrees
- moved R8 359.0 mm to (409.5, 399.9)
- moved Q4 356.6 mm to (421.3, 400.9), turned to 0 degrees
- moved ROUT1 354.4 mm to (409.5, 416.1), turned to 0 degrees
- moved D4 349.8 mm to (425.7, 397.8), turned to 0 degrees
- moved R9 349.1 mm to (409.5, 403.9), turned to 0 degrees
- moved TP3 345.8 mm to (447.9, 451.2), turned to 0 degrees
- moved R7 344.1 mm to (409.5, 395.8), turned to 0 degrees
- moved R3 343.7 mm to (403.8, 320.9)
- moved R1 341.6 mm to (409.5, 391.8), turned to 0 degrees
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- renumbered TP_tierra1 to TP17, TP_tierra2 to TP18
