File: Prototipo_/Prototipo/prototipo.kicad_pcb (KiCad board)
At the start: 2 copper layers, 124 parts, among them J1 Conn_01x02_Socket, J4 Conn_01x12_Pin, Q1 MMBT2222A, Q10 MMBT2222A, Q11 MMBT2907A, Q12 MMBT2222A, Q13 MMBT2222A, Q14 MMBT2907A, Q15 MMBT2222A, Q16 MMBT2222A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

Commit message: pruebo modulos de celdas en el esquematico del pcb
Parts:
- removed J4: Conn_01x12_Pin, Connector_PinHeader_2.54mm:PinHeader_1x12_P2.54mm_Vertical
- removed TP10, TP11, TP12, TP13, TP14, TP15, TP16, TP3, TP4, TP5, TP6, TP7, TP8, TP9, TP_tierra1, TP_tierra2: TestPoint, TestPoint:TestPoint_Bridge_Pitch2.54mm_Drill1.0mm
- added J2: Conn_01x06_Pin, Connector_JST:JST_VH_B6P-VH-B_1x06_P3.96mm_Vertical, F.Cu at (313.5, 307.0)
- added J3: Conn_01x06_Pin, Connector_JST:JST_VH_B6P-VH-B_1x06_P3.96mm_Vertical, F.Cu at (312.0, 231.1)
- moved VCELL1 402.3 mm to (401.2, 374.0)
- moved VCELL2 386.8 mm to (405.7, 303.0)
- moved Q3 358.0 mm to (411.1, 392.4), turned to 0 degrees
- moved Q1 352.1 mm to (411.1, 388.0), turned to 0 degrees
- moved R8 352.1 mm to (399.3, 395.9)
- moved Q4 349.5 mm to (411.1, 396.9), turned to 0 degrees
- moved ROUT1 347.0 mm to (399.3, 412.1), turned to 0 degrees
- moved A1 345.2 mm to (536.0, 275.5), turned to 180 degrees
- moved R3 343.7 mm to (403.8, 320.9)
- moved D4 342.5 mm to (415.5, 393.8), turned to 0 degrees
- moved R9 341.8 mm to (399.3, 399.9), turned to 0 degrees
- moved S2 339.6 mm to (421.3, 318.7), turned to 0 degrees
- moved Q7 339.3 mm to (415.5, 321.5), turned to 0 degrees
- moved R7 336.6 mm to (399.3, 391.8), turned to 0 degrees
- moved R1 335.0 mm to (399.3, 387.8), turned to 0 degrees
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