File: Prototipo_/Prototipo/prototipo_nuevo.kicad_sch (KiCad schematic)
At the start: 13 parts, among them J1 Conn_01x02_Socket, J4 Conn_01x12_Pin

Commit message: pruebo modulos de celdas en el esquematico del pcb
Parts:
- removed J4: Conn_01x12_Pin, Connector_PinHeader_2.54mm:PinHeader_1x12_P2.54mm_Vertical, symbol Connector:Conn_01x12_Pin
- removed TP15, TP16, TP_tierra1, TP_tierra2: TestPoint, TestPoint:TestPoint_Bridge_Pitch2.54mm_Drill1.0mm, symbol Connector:TestPoint
- added J2, J3: Conn_01x06_Pin, Connector_JST:JST_VH_B6P-VH-B_1x06_P3.96mm_Vertical, symbol Connector:Conn_01x06_Pin
- renumbered SGND1 to SGND12
Connections:
- net GND: now also J2.1 (Pin_1)
- net VCC: now also J2.2 (Pin_2)
- net Vc1: now also J2.5 (Pin_5)
- net Vc2: now also J3.3 (Pin_3)
- net Vc21: now also J3.1 (Pin_1)
- net Vc22: now also J3.2 (Pin_2)
- net Vc3: now also J3.6 (Pin_6)
- net Vc31: now also J3.4 (Pin_4)
- net Vc32: now also J3.5 (Pin_5)
- net Vc_11: now also J2.3 (Pin_3)
- net Vc_12: now also J2.4 (Pin_4)
