File: Prototipo_/Prototipo/switch_banco.kicad_sch (KiCad schematic)
At the start: 7 parts

Commit message: pruebo modulos de celdas en el esquematico del pcb
Parts:
- renumbered D_B1 to D1, QB_1 to Q1_1, QB_2 to Q1_2, RB_2 to R1_7, RB_3 to R1_8, RB_1 to R1_9, SB_1 to S1
Changed lines of the file:
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@@
 		(on_board yes)
 		(dnp no)
-		(property "Reference" "SB_1"
+		(property "Reference" "S1"
 			(at 95.885 93.98 0)
 			(effects
@@
 			(project "prototipo"
 				(path "/c9225433-a7fd-41e8-8162-e91e829dcb79/69120eb2-13db-48bd-9e77-f62722c18bbc"
-					(reference "SB_3")
+					(reference "S3")
 					(unit 1)
 				)
 				(path "/c9225433-a7fd-41e8-8162-e91e829dcb79/7c9a14ee-10ad-4ddf-af17-6bfeb468e011"
-					(reference "SB_1")
+					(reference "S1")
 					(unit 1)
 				)
 				(path "/c9225433-a7fd-41e8-8162-e91e829dcb79/aa26f19e-f2c7-49c1-961b-509062eddf74"
-					(reference "SB_2")
+					(reference "S2")
 					(unit 1)
 				)
@@
 		(on_board yes)
 		(dnp no)
-		(property "Reference" "RB_3"
+		(property "Reference" "R1_8"
 			(at 127.3302 94.615 0)
 			(effects
@@
 			(project "prototipo"
 				(path "/c9225433-a7fd-41e8-8162-e91e829dcb79/69120eb2-13db-48bd-9e77-f62722c18bbc"
-					(reference "RB_9")
+					(reference "R3_8")
 					(unit 1)
 				)
 				(path "/c9225433-a7fd-41e8-8162-e91e829dcb79/7c9a14ee-10ad-4ddf-af17-6bfeb468e011"
-					(reference "RB_3")
+					(reference "R1_8")
 					(unit 1)
 				)
 				(path "/c9225433-a7fd-41e8-8162-e91e829dcb79/aa26f19e-f2c7-49c1-961b-509062eddf74"
-					(reference "RB_6")
+					(reference "R2_8")
 					(unit 1)
 				)
@@
 		(on_board yes)
 		(dnp no)
-		(property "Reference" "QB_1"
+		(property "Reference" "Q1_1"
 			(at 125.095 106.68 0)
 			(effects
@@
 			(project "prototipo"
 				(path "/c9225433-a7fd-41e8-8162-e91e829dcb79/69120eb2-13db-48bd-9e77-f62722c18bbc"
-					(reference "QB_5")
+					(reference "Q3_1")
 					(unit 1)
 				)
 				(path "/c9225433-a7fd-41e8-8162-e91e829dcb79/7c9a14ee-10ad-4ddf-af17-6bfeb468e011"
-					(reference "QB_1")
+					(reference "Q1_1")
 					(unit 1)
 				)
 				(path "/c9225433-a7fd-41e8-8162-e91e829dcb79/aa26f19e-f2c7-49c1-961b-509062eddf74"
-					(reference "QB_3")
+					(reference "Q2_1")
 					(unit 1)
 				)
@@
 		(on_board yes)
 		(dnp no)
-		(property "Reference" "QB_2"
+		(property "Reference" "Q1_2"
 			(at 142.875 68.58 0)
 			(effects
@@
 			(project "prototipo"
 				(path "/c9225433-a7fd-41e8-8162-e91e829dcb79/69120eb2-13db-48bd-9e77-f62722c18bbc"
-					(reference "QB_6")
+					(reference "Q3_2")
 					(unit 1)
 				)
 				(path "/c9225433-a7fd-41e8-8162-e91e829dcb79/7c9a14ee-10ad-4ddf-af17-6bfeb468e011"
-					(reference "QB_2")
+					(reference "Q1_2")
 					(unit 1)
 				)
 				(path "/c9225433-a7fd-41e8-8162-e91e829dcb79/aa26f19e-f2c7-49c1-961b-509062eddf74"
-					(reference "QB_4")
+					(reference "Q2_2")
 					(unit 1)
 				)
@@
 		(on_board yes)
 		(dnp no)
-		(property "Reference" "RB_1"
+		(property "Reference" "R1_9"
 			(at 111.125 106.68 90)
 			(effects
@@
 			(project "prototipo"
 				(path "/c9225433-a7fd-41e8-8162-e91e829dcb79/69120eb2-13db-48bd-9e77-f62722c18bbc"
-					(reference "RB_7")
+					(reference "R3_9")
 					(unit 1)
 				)
 				(path "/c9225433-a7fd-41e8-8162-e91e829dcb79/7c9a14ee-10ad-4ddf-af17-6bfeb468e011"
-					(reference "RB_1")
+					(reference "R1_9")
 					(unit 1)
 				)
 				(path "/c9225433-a7fd-41e8-8162-e91e829dcb79/aa26f19e-f2c7-49c1-961b-509062eddf74"
-					(reference "RB_4")
+					(reference "R2_9")
 					(unit 1)
 				)
@@
 		(on_board yes)
 		(dnp no)
-		(property "Reference" "RB_2"
+		(property "Reference" "R1_7"
 			(at 127.3302 67.945 0)
 			(effects
@@
 			(project "prototipo"
 				(path "/c9225433-a7fd-41e8-8162-e91e829dcb79/69120eb2-13db-48bd-9e77-f62722c18bbc"
-					(reference "RB_8")
+					(reference "R3_7")
 					(unit 1)
 				)
 				(path "/c9225433-a7fd-41e8-8162-e91e829dcb79/7c9a14ee-10ad-4ddf-af17-6bfeb468e011"
-					(reference "RB_2")
+					(reference "R1_7")
 					(unit 1)
 				)
 				(path "/c9225433-a7fd-41e8-8162-e91e829dcb79/aa26f19e-f2c7-49c1-961b-509062eddf74"
-					(reference "RB_5")
+					(reference "R2_7")
 					(unit 1)
 				)
@@
 		(on_board yes)
 		(dnp no)
-		(property "Reference" "D_B1"
+		(property "Reference" "D1"
 			(at 112.395 69.85 0)
 			(effects
@@
 			(project "prototipo"
 				(path "/c9225433-a7fd-41e8-8162-e91e829dcb79/69120eb2-13db-48bd-9e77-f62722c18bbc"
-					(reference "D_B3")
+					(reference "D3")
 					(unit 1)
 				)
 				(path "/c9225433-a7fd-41e8-8162-e91e829dcb79/7c9a14ee-10ad-4ddf-af17-6bfeb468e011"
-					(reference "D_B1")
+					(reference "D1")
 					(unit 1)
 				)
 				(path "/c9225433-a7fd-41e8-8162-e91e829dcb79/aa26f19e-f2c7-49c1-961b-509062eddf74"
-					(reference "D_B2")
-					(unit 1)
-				)
+					(reference "D2")
+					(unit 1)
+				)
