File: Prototipo/Prototipo/prototipo.kicad_sch (KiCad schematic)
At the start: 10 parts, among them J1 Conn_01x02_Socket, J2 Conn_01x06_Pin, J3 Conn_01x06_Pin

Commit message: propuesta de disposición de los elementos del pcb
subo antes de empezar a hacer el ruteo
Parts:
- removed J2, J3: Conn_01x06_Pin, Connector_JST:JST_VH_B6P-VH-B_1x06_P3.96mm_Vertical, symbol Connector:Conn_01x06_Pin
- added J4: Conn_01x12_Pin, Connector_PinHeader_2.54mm:PinHeader_1x12_P2.54mm_Vertical, symbol Connector:Conn_01x12_Pin
- added TP_tierra1, TP_tierra2, TP_tierra3, TP_tierra4: TestPoint, TestPoint:TestPoint_Bridge_Pitch2.54mm_Drill1.0mm, symbol Connector:TestPoint
- J_B1, J_B2: footprint Connector_JST:JST_VH_B2P-VH_1x02_P3.96mm_Vertical -> Connector_PinHeader_2.54mm:PinHeader_1x02_P2.54mm_Vertical
- renumbered SGND12 to SGND1
Connections:
- net 0: now also TP_tierra1.1, TP_tierra2.1, TP_tierra3.1, TP_tierra4.1
- net GND: now also J4.1 (Pin_1), J4.12 (Pin_12)
- net VCC: now also J4.2 (Pin_2)
- net Vc1: now also J4.9 (Pin_9)
- net Vc2: now also J4.10 (Pin_10)
- net Vc3: now also J4.11 (Pin_11)
- net Vc_11: now also A1.1, J4.3 (Pin_3); no longer A1.13
- net Vc_12: now also A1.13, J4.6 (Pin_6); no longer A1.1
- net Vc_21: now also A1.3, J4.4 (Pin_4); no longer A1.11
- net Vc_22: now also A1.11, J4.7 (Pin_7); no longer A1.3
- net Vc_31: now also A1.5, J4.5 (Pin_5); no longer A1.9
- net Vc_32: now also A1.9, J4.8 (Pin_8); no longer A1.5
- net celda_1/Vcontrol_neg: now also A1.2; no longer A1.12
- net celda_2/Vcontrol_neg: now also A1.12; no longer A1.2
- net celda_3/Vcontrol_neg: now also A1.4; no longer A1.10
- net celda_4/Vcontrol_neg: now also A1.10; no longer A1.4
- net celda_5/Vcontrol_neg: now also A1.6; no longer A1.8
- net celda_6/Vcontrol_neg: now also A1.8; no longer A1.6
