File: Prototipo/Prototipo/prototipo.kicad_pcb (KiCad board)
At the start: 2 copper layers, 124 parts, among them J1 Conn_01x02_Socket, J4 Conn_01x12_Pin, Q1 MMBT2222A, Q10 MMBT2222A, Q11 MMBT2907A, Q12 MMBT2222A, Q13 MMBT2222A, Q14 MMBT2907A, Q15 MMBT2222A, Q16 MMBT2222A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

Commit message: propuesta de disposición de los elementos del pcb
subo antes de empezar a hacer el ruteo
Parts:
- J_B1, J_B2: footprint Connector_JST:JST_VH_B2P-VH_1x02_P3.96mm_Vertical -> Connector_PinHeader_2.54mm:PinHeader_1x02_P2.54mm_Vertical
- moved TP_tierra2 324.8 mm to (292.4, 286.0)
- moved R30 301.0 mm to (700.5, 285.5), turned to 180 degrees
- moved VCELL5 295.4 mm to (658.9, 307.5)
- moved SGND1 288.4 mm to (482.6, 159.0)
- moved S5 283.4 mm to (724.5, 287.5), turned to 90 degrees
- moved R29 282.5 mm to (692.9, 291.0)
- moved R26 280.7 mm to (677.5, 284.8), turned to 90 degrees
- moved R28 280.2 mm to (698.1, 279.8), turned to 90 degrees
- moved TP7 279.7 mm to (705.6, 268.0), turned to 90 degrees
- moved Q15 277.6 mm to (693.0, 281.5), turned to -90 degrees
- moved ROUT5 277.1 mm to (673.3, 284.5), turned to 180 degrees
- moved D5 268.0 mm to (700.5, 268.0), turned to 180 degrees
- moved Q14 264.8 mm to (685.7, 280.1)
- moved Q13 257.8 mm to (685.6, 263.0), turned to -90 degrees
- moved VCELL6 255.8 mm to (730.2, 140.0), turned to 180 degrees
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- renumbered TP17 to TP_tierra1, TP18 to TP_tierra2, TP16 to TP_tierra3, TP15 to TP_tierra4, VCELL3 to VCELL2, VCELL2 to VCELL3
Connections:
- A1 pad 1: Vc_12 -> Vc_11
- A1 pad 10: /celda_3/Vcontrol_neg -> /celda_4/Vcontrol_neg
- A1 pad 11: Vc_21 -> Vc_22
- A1 pad 12: /celda_1/Vcontrol_neg -> /celda_2/Vcontrol_neg
- A1 pad 13: Vc_11 -> Vc_12
- A1 pad 2: /celda_2/Vcontrol_neg -> /celda_1/Vcontrol_neg
- A1 pad 3: Vc_22 -> Vc_21
- A1 pad 4: /celda_4/Vcontrol_neg -> /celda_3/Vcontrol_neg
- A1 pad 5: Vc_32 -> Vc_31
- A1 pad 6: /celda_6/Vcontrol_neg -> /celda_5/Vcontrol_neg
- A1 pad 8: /celda_5/Vcontrol_neg -> /celda_6/Vcontrol_neg
- A1 pad 9: Vc_31 -> Vc_32
- J4 pad 10: Vc31 -> Vc2
- J4 pad 11: Vc32 -> Vc3
- J4 pad 12: Vc3 -> GND
- J4 pad 2: GND -> VCC
- J4 pad 3: VCC -> Vc_11
- J4 pad 4: Vc_11 -> Vc_21
- J4 pad 5: Vc_12 -> Vc_31
- J4 pad 6: Vc1 -> Vc_12
- J4 pad 7: Vc21 -> Vc_22
- J4 pad 8: Vc22 -> Vc_32
- J4 pad 9: Vc2 -> Vc1

Commit message: propuesta de ruteo de celdas
solo el ruteo de las celdas, falta el general
Parts:
- moved TP2 97.7 mm to (631.5, 264.5)
- moved TP14 15.7 mm to (702.7, 174.0), turned to 180 degrees
- moved TP1 15.5 mm to (535.7, 263.5)
- moved VCELL6 15.5 mm to (714.8, 139.5)
- moved S6 15.0 mm to (649.7, 159.5)
- moved TP8 10.4 mm to (673.2, 178.5), turned to 0 degrees
- moved TP12 9.80 mm to (621.0, 174.0), turned to 180 degrees
- moved Q16 9.20 mm to (694.7, 183.5)
- moved VCELL4 9.00 mm to (633.1, 139.5)
- moved ROUT6 8.89 mm to (707.1, 162.0)
- moved R33 8.89 mm to (694.7, 171.2)
- moved Q18 8.89 mm to (687.4, 165.0)
- moved R35 8.89 mm to (687.5, 155.5)
- moved R36 8.89 mm to (679.9, 161.0)
- moved R34 8.89 mm to (682.2, 166.7), turned to 180 degrees
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Routing:
- net /celda_3/bus_pos: track 0.00 -> 195.3 mm
- net /celda_5/bus_pos: track 0.00 -> 193.2 mm
- net /celda_1/bus_pos: track 0.00 -> 188.3 mm
- net Net-(J1-Pin_1): track 0.00 -> 95.1 mm
- net /celda_2/gate: track 0.00 -> 68.7 mm
- net /celda_3/gate: track 0.00 -> 68.7 mm
- net /celda_1/gate: track 0.00 -> 68.7 mm
- net /celda_4/gate: track 0.00 -> 60.7 mm
- net /celda_6/gate: track 0.00 -> 60.7 mm
- net /celda_5/gate: track 0.00 -> 55.1 mm
- net Net-(D_B3-+): track 0.00 -> 40.2 mm
- net Net-(D_B2-+): track 0.00 -> 40.2 mm
- net Net-(D_B1-+): track 0.00 -> 39.2 mm
- net /celda_2/cell_neg: track 0.00 -> 33.6 mm
- net /celda_3/cell_neg: track 0.00 -> 33.6 mm
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Other:
- board text added: "${REFERENCE}"
