File: Prototipo/prototipo.kicad_pcb (KiCad board)
At the start: 2 copper layers, 124 parts, among them J1 Conn_01x02_Socket, J4 Conn_01x12_Pin, Q1 MMBT2222A, Q10 MMBT2222A, Q11 MMBT2907A, Q12 MMBT2222A, Q13 MMBT2222A, Q14 MMBT2907A, Q15 MMBT2222A, Q16 MMBT2222A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

Commit message: subo listita de materiales del prototipo
Parts:
- moved R6 9.39 mm to (600.0, 293.0)
- moved R29 9.39 mm to (683.7, 293.0)
- moved R25 9.37 mm to (677.3, 257.0)
- moved D5 9.29 mm to (691.3, 269.5)
- moved D_B3 9.29 mm to (713.8, 270.7)
- moved Q8 9.29 mm to (600.1, 283.0)
- moved QB_5 9.29 mm to (690.3, 258.4)
- moved R3 9.29 mm to (584.6, 286.0)
- moved R30 9.29 mm to (691.3, 287.0)
- moved RB_5 9.29 mm to (619.6, 260.0)
- moved RB_6 9.29 mm to (612.1, 254.5)
- moved RB_7 9.29 mm to (684.8, 259.6)
- moved VCELL3 9.29 mm to (572.7, 308.5)
- moved D2 9.29 mm to (607.6, 269.5)
- moved D_B2 9.29 mm to (629.9, 271.0)
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Routing:
- net /celda_3/gate: track 68.7 -> 61.3 mm
- net /celda_5/gate: track 55.1 -> 61.3 mm
- net /celda_3/cell_neg: track 33.6 -> 28.3 mm
- net /celda_5/cell_neg: track 33.6 -> 28.3 mm
- net Net-(Q2-B): track 3.88 -> 6.52 mm
- net Net-(Q13-B): track 3.88 -> 6.47 mm
- net Net-(Q1-B): track 3.88 -> 6.45 mm
- net Net-(Q10-B): track 3.88 -> 6.45 mm
- net Net-(Q16-B): track 3.88 -> 6.45 mm
- net Net-(Q6-B): track 3.88 -> 5.92 mm
- net /celda_1/gate: track 68.7 -> 69.8 mm
- net Net-(Q3-C): track 12.8 -> 13.8 mm
- net Net-(Q5-C): track 12.8 -> 13.8 mm
- net /celda_2/gate: track 68.7 -> 69.7 mm
- net /celda_6/gate: track 60.7 -> 61.3 mm
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
Commit message: actualizo el listadito de compras
Parts:
- moved J4 96.0 mm to (487.5, 204.1)
- moved A1 94.2 mm to (494.3, 206.6)
- moved J_B2 19.8 mm to (702.9, 263.5)
- moved J_B1 15.6 mm to (618.9, 263.8)
- moved D_B1 13.0 mm to (542.3, 282.1)
- moved D_B2 13.0 mm to (626.3, 283.6)
- moved Q13 13.0 mm to (672.9, 277.0)
- moved Q14 13.0 mm to (671.9, 294.5)
- moved Q15 13.0 mm to (680.2, 295.5)
- moved Q4 13.0 mm to (512.2, 295.0)
- moved Q6 13.0 mm to (589.1, 277.0)
- moved Q7 13.0 mm to (588.1, 294.5)
- moved QB_1 13.0 mm to (518.8, 269.7)
- moved QB_3 13.0 mm to (602.8, 271.2)
- moved R1 13.0 mm to (512.1, 305.5)
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Routing:
- net Net-(J1-Pin_1): track 95.1 -> 0.00 mm
- net Vc_31: track 0.00 -> 36.6 mm
- net Vc_32: track 0.00 -> 26.9 mm
- net Vc_21: track 0.00 -> 26.7 mm
- net Vc_22: track 0.00 -> 21.8 mm
- net Vc_11: track 0.00 -> 16.0 mm
- net Vc_12: track 0.00 -> 14.9 mm
- net /celda_5/bus_pos: track 193.2 -> 178.4 mm
- net VCC: track 0.00 -> 7.87 mm
- net /celda_3/bus_pos: track 195.0 -> 188.7 mm

Commit message: Aplicar gitignore y dejar de trackear archivos innecesarios
Parts:
- removed QB_4: MMBFJ201, Package_TO_SOT_SMD:SOT-23-3
- added F1: Fuse, Fuse:Fuseholder_Cylinder-5x20mm_Schurter_0031_8201_Horizontal_Open, F.Cu at (514.7, 314.5)
- added F2: Fuse, Fuse:Fuseholder_Cylinder-5x20mm_Schurter_0031_8201_Horizontal_Open, F.Cu at (610.5, 319.0)
- added F3: Fuse, Fuse:Fuseholder_Cylinder-5x20mm_Schurter_0031_8201_Horizontal_Open, F.Cu at (761.2, 180.8)
- added F4: Fuse, Fuse:Fuseholder_Cylinder-5x20mm_Schurter_0031_8201_Horizontal_Open, F.Cu at (790.2, 167.7)
- added F5: Fuse, Fuse:Fuseholder_Cylinder-5x20mm_Schurter_0031_8201_Horizontal_Open, F.Cu at (711.9, 274.5)
- added F6: Fuse, Fuse:Fuseholder_Cylinder-5x20mm_Schurter_0031_8201_Horizontal_Open, F.Cu at (761.2, 167.7)
- SB_1, SB_2, SB_3: value AO3401A -> FDMS6681Z; footprint Package_TO_SOT_SMD:SOT-23-3 -> Package_TO_SOT_SMD:PQFN_8x8
- VCELL1, VCELL2, VCELL3, VCELL4, VCELL5, VCELL6: moved to B.Cu
- moved TP_tierra1 139.1 mm to (402.7, 216.2)
- moved TP_tierra2 139.1 mm to (412.7, 216.0)
- moved TP_tierra3 139.1 mm to (426.0, 216.0)
- moved TP_tierra4 139.1 mm to (439.0, 216.0)
- moved A1 72.6 mm to (564.9, 189.6)
- moved VCELL5 52.2 mm to (644.3, 269.5)
- moved S5 45.4 mm to (717.9, 255.6)
- moved SGND11 40.5 mm to (520.7, 284.5)
- moved VCELL1 39.3 mm to (447.1, 309.5)
- moved SB_1 38.8 mm to (502.6, 303.0)
- moved R12 36.9 mm to (485.8, 313.5)
- moved QB_2 36.2 mm to (497.4, 276.9)
- moved R10 36.2 mm to (483.4, 305.8)
- moved RB_3 36.2 mm to (490.6, 278.0)
- moved TP3 36.2 mm to (492.4, 294.0)
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Connections:
- S1 pad 2: /celda_1/bus_neg -> Net-(S1-D)
- S2 pad 2: /celda_1/bus_pos -> Net-(S2-D)
- S3 pad 2: /celda_1/bus_pos -> Net-(S3-D)
- S4 pad 2: /celda_1/bus_neg -> Net-(S4-D)
- S5 pad 2: /celda_3/bus_pos -> Net-(S5-D)
- S6 pad 2: /celda_3/bus_pos -> Net-(S6-D)
Routing:
- net Net-(D_B3-+): track 40.2 -> 0.00 mm
- net /celda_3/bus_pos: track 188.7 -> 152.0 mm
- net Vc_31: track 36.6 -> 0.00 mm
- net /celda_5/bus_pos: track 178.4 -> 143.0 mm
- net /celda_5/gate: track 61.3 -> 31.0 mm
- net /celda_3/gate: track 61.3 -> 31.0 mm
- net Net-(D_B2-+): track 40.2 -> 10.1 mm
- net Vc_32: track 26.9 -> 0.00 mm
- net Vc_21: track 26.7 -> 0.00 mm
- net /celda_1/gate: track 69.8 -> 44.6 mm
- net Net-(S2-D): track 0.00 -> 25.2 mm
- net Vc_12: track 14.9 -> 39.4 mm
- net Net-(VCELL5-+): track 22.5 -> 0.11 mm
- net Net-(VCELL1-+): track 22.5 -> 0.11 mm
- net Vc_22: track 21.8 -> 0.00 mm
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Other:
- board text removed: "${REFERENCE}"

Commit message: Cambios de prototipo con el nuevo pmos
Parts:
- added QB_4: MMBFJ201, Package_TO_SOT_SMD:SOT-23-3, F.Cu at (571.0, 273.5)
- added TP15: TestPoint, TestPoint:TestPoint_Bridge_Pitch2.54mm_Drill1.0mm, F.Cu at (470.0, 262.5)
- added TP16: TestPoint, TestPoint:TestPoint_Bridge_Pitch2.54mm_Drill1.0mm, F.Cu at (578.5, 267.5)
- added TP17: TestPoint, TestPoint:TestPoint_Bridge_Pitch2.54mm_Drill1.0mm, F.Cu at (714.5, 244.5)
- added TP18: TestPoint, TestPoint:TestPoint_Bridge_Pitch2.54mm_Drill1.0mm, F.Cu at (513.5, 292.5)
- added TP19: TestPoint, TestPoint:TestPoint_Bridge_Pitch2.54mm_Drill1.0mm, F.Cu at (622.0, 321.0)
- added TP20: TestPoint, TestPoint:TestPoint_Bridge_Pitch2.54mm_Drill1.0mm, F.Cu at (444.5, 126.5)
- added TP21: TestPoint, TestPoint:TestPoint_Bridge_Pitch2.54mm_Drill1.0mm, F.Cu at (572.0, 138.5)
- added TP22: TestPoint, TestPoint:TestPoint_Bridge_Pitch2.54mm_Drill1.0mm, F.Cu at (707.5, 241.5)
- added TP23: TestPoint, TestPoint:TestPoint_Bridge_Pitch2.54mm_Drill1.0mm, F.Cu at (658.0, 139.5)
- moved F3 283.5 mm to (483.8, 122.5)
- moved F4 247.1 mm to (549.5, 112.0)
- moved F6 147.0 mm to (623.0, 117.5)
Routing:
- net /celda_1/cell_neg: track 30.9 -> 39.6 mm
- net /celda_5/cell_neg: track 30.9 -> 22.9 mm
- net /celda_1/gate: track 44.6 -> 47.1 mm
- net /celda_1/bus_pos: track 187.3 -> 189.8 mm

Commit message: ruteado de celda uno
Parts:
- moved TP2 53.4 mm to (545.5, 316.5)
- moved R28 48.4 mm to (657.8, 308.5), turned to 0 degrees
- moved Q15 48.1 mm to (652.1, 309.5)
- moved TP19 46.8 mm to (595.3, 282.5), turned to 90 degrees
- moved D5 45.5 mm to (662.3, 294.5)
- moved F5 45.5 mm to (691.3, 315.0)
- moved Q13 45.5 mm to (647.5, 289.5)
- moved Q14 45.5 mm to (646.5, 307.0)
- moved R25 45.5 mm to (648.5, 282.0)
- moved R26 45.5 mm to (639.4, 311.0)
- moved R27 45.5 mm to (647.5, 301.8)
- moved R29 45.5 mm to (654.8, 318.5)
- moved R30 45.5 mm to (662.3, 314.0)
- moved ROUT5 45.5 mm to (635.2, 311.0)
- moved TP13 45.5 mm to (639.5, 299.0)
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Routing:
- net /celda_3/gate: track 31.0 -> 99.2 mm
- net /celda_1/gate: track 47.1 -> 114.2 mm
- net Net-(D_B3-+): track 0.00 -> 48.1 mm
- net Net-(S4-D): track 0.00 -> 41.8 mm
- net Net-(S5-D): track 0.00 -> 41.8 mm
- net Net-(D_B2-+): track 10.1 -> 48.1 mm
- net /celda_5/gate: track 31.0 -> 62.5 mm
- net Net-(QB_5-C): track 0.00 -> 21.1 mm
- net /celda_1/bus_neg: track 0.00 -> 18.9 mm
- net Net-(S2-D): track 25.2 -> 41.8 mm
- net /celda_3/bus_pos: track 152.0 -> 168.0 mm
- net /celda_3/cell_neg: track 20.7 -> 32.3 mm
- net Net-(VCELL1-+): track 0.11 -> 11.2 mm
- net Net-(VCELL5-+): track 0.11 -> 11.2 mm
- net Net-(D_B1-+): track 37.2 -> 48.1 mm
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
Commit message: ruteo de un banco
Parts:
- removed SB_2, SB_3: FDMS6681Z, Package_TO_SOT_SMD:PQFN_8x8
- added Q20: FDMS6681Z, Huellas:FDMS6681Z, F.Cu at (688.5, 302.4)
- added Q21: FDMS6681Z, Huellas:FDMS6681Z, F.Cu at (591.0, 303.4)
- SB_1: footprint Package_TO_SOT_SMD:PQFN_8x8 -> Huellas:FDMS6681Z
- VCELL1, VCELL2, VCELL3, VCELL4, VCELL5, VCELL6: footprint Battery:BatteryHolder_MPD_BK-18650-PC2 -> Huellas:BatteryHolder_MPD_BK-18650-PC2
- moved TP20 130.4 mm to (452.5, 256.6)
- moved S1 130.3 mm to (451.7, 272.6), turned to 0 degrees
- moved SGND1 126.0 mm to (462.7, 272.6), turned to 0 degrees
- moved F3 124.6 mm to (452.2, 243.0)
- moved Q5 104.0 mm to (497.0, 251.0)
- moved R15 104.0 mm to (496.0, 256.2), turned to 180 degrees
- moved R14 104.0 mm to (504.1, 247.0)
- moved ROUT3 104.0 mm to (508.3, 247.0)
- moved R17 104.0 mm to (488.7, 239.5)
- moved TP11 102.4 mm to (501.3, 256.2)
- moved R18 102.1 mm to (481.1, 244.0)
- moved Q2 100.2 mm to (488.4, 260.8)
- moved R16 98.5 mm to (512.4, 253.2), turned to -90 degrees
- moved VCELL2 96.8 mm to (519.8, 256.5)
- moved R13 95.3 mm to (494.9, 265.3), turned to 0 degrees
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Connections:
- SB_1 pad 1: Net-(D_B1-+) -> /celda_1/bus_pos
- SB_1 pad 3: /celda_1/bus_neg -> /celda_1/bus_pos
Routing:
- net /celda_5/gate: track 62.5 -> 104.3 mm
- net Vc_12: track 39.4 -> 0.00 mm
- net Net-(S1-D): track 0.00 -> 36.8 mm
- net /celda_1/bus_pos: track 196.5 -> 162.1 mm
- net /celda_1/bus_neg: track 18.9 -> 53.1 mm
- net /celda_2/gate: track 69.7 -> 100.5 mm
- net Net-(Q9-C): track 2.93 -> 21.6 mm
- net /celda_5/bus_pos: track 151.5 -> 133.6 mm
- net Net-(Q9-B): track 4.43 -> 22.1 mm
- net Net-(Q4-B): track 4.80 -> 22.1 mm
- net Net-(Q4-C): track 4.68 -> 21.6 mm
- net /celda_1/gate: track 114.2 -> 98.7 mm
- net Net-(Q1-C): track 3.55 -> 14.3 mm
- net Net-(Q2-B): track 16.8 -> 8.84 mm
- net Net-(D_B1-+): track 48.1 -> 40.4 mm
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
Commit message: ruteo de dos celdas más
Chequear la orientación de los portapilas
Parts:
- moved A1 178.0 mm to (362.3, 288.6)
- moved Q20 115.6 mm to (575.6, 277.3), turned to 90 degrees
- moved Q21 73.6 mm to (659.5, 276.4), turned to 90 degrees
- moved TP2 65.7 mm to (594.1, 274.4), turned to -90 degrees
- moved R28 42.1 mm to (615.9, 304.8), turned to 90 degrees
- moved R5 26.3 mm to (535.6, 304.7), turned to 90 degrees
- moved Q15 25.1 mm to (628.0, 316.4), turned to 90 degrees
- moved QB_6 23.7 mm to (660.3, 295.4), turned to 0 degrees
- moved QB_4 23.1 mm to (576.5, 296.3), turned to 0 degrees
- moved TP22 22.9 mm to (675.3, 300.9), turned to 180 degrees
- moved D5 20.2 mm to (647.7, 308.5)
- moved TP7 19.5 mm to (655.4, 307.0)
- moved QB_3 18.0 mm to (569.7, 295.8)
- moved D_B3 17.9 mm to (669.8, 284.7), turned to -90 degrees
- moved QB_5 15.6 mm to (653.5, 294.9)
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Routing:
- net /celda_3/bus_pos: track 162.2 -> 243.1 mm, vias 0 -> 4
- net Net-(J1-Pin_1): track 0.00 -> 79.0 mm
- net /celda_1/bus_pos: track 162.1 -> 236.3 mm, vias 0 -> 4
- net /celda_5/bus_pos: track 133.6 -> 182.6 mm, vias 0 -> 4
- net /celda_1/bus_neg: track 53.1 -> 97.5 mm
- net /celda_5/gate: track 104.3 -> 85.5 mm
- net /celda_3/gate: track 104.2 -> 86.6 mm
- net Net-(Q15-B): track 4.80 -> 22.1 mm
- net Net-(Q8-B): track 4.80 -> 22.1 mm
- net Net-(Q15-C): track 4.68 -> 21.6 mm
- net Net-(Q8-C): track 4.68 -> 21.6 mm
- net Net-(Q6-C): track 3.55 -> 14.3 mm
- net Net-(Q13-C): track 3.55 -> 14.3 mm
- net Net-(D_B2-+): track 48.1 -> 40.4 mm
- net Net-(D_B3-+): track 48.1 -> 40.4 mm
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
Commit message: cambio el zener y subo la listita de compras
Parts:
- F1, F2, F3, F4, F5, F6: footprint Fuse:Fuseholder_Cylinder-5x20mm_Schurter_0031_8201_Horizontal_Open -> Huellas:Fuseholder_Cylinder-5x20mm_Schurter_0031_8201_Horizontal_Open
- J1: footprint TerminalBlock:TerminalBlock_MaiXu_MX126-5.0-02P_1x02_P5.00mm -> Huellas:TerminalBlock_bornier-2_P5.08mm
- moved TP_tierra1 188.6 mm to (516.8, 229.2)
- moved TP_tierra2 188.6 mm to (526.7, 229.0)
- moved TP_tierra3 188.6 mm to (540.0, 229.0)
- moved TP_tierra4 188.6 mm to (553.0, 229.0)
- moved F4 132.0 mm to (533.3, 243.0)
- moved S6 131.2 mm to (612.6, 272.6), turned to 0 degrees
- moved S3 130.7 mm to (532.7, 272.6), turned to 0 degrees
- moved F6 125.9 mm to (613.1, 243.0)
- moved TP23 125.4 mm to (613.4, 256.6)
- moved TP21 124.3 mm to (533.5, 256.6)
- moved Q17 105.1 mm to (657.9, 251.0)
- moved R33 105.1 mm to (656.9, 256.2), turned to 180 degrees
- moved R32 105.1 mm to (665.0, 247.0)
- moved ROUT6 105.1 mm to (669.2, 247.0)
- moved R35 104.7 mm to (649.6, 239.5)
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Connections:
- A1 pad 7: GND -> 0
- J4 pad 1: GND -> 0
- J4 pad 12: GND -> 0
Routing:
- net /celda_3/bus_pos: track 243.1 -> 327.5 mm
- net Net-(S6-D): track 0.00 -> 36.8 mm
- net Net-(S3-D): track 0.00 -> 36.8 mm
- net /celda_4/gate: track 61.2 -> 89.1 mm
- net /celda_6/gate: track 61.3 -> 88.1 mm
- net Net-(Q18-C): track 2.93 -> 21.7 mm
- net Net-(Q12-C): track 2.93 -> 21.7 mm
- net Net-(Q18-B): track 4.43 -> 22.1 mm
- net Net-(Q12-B): track 4.43 -> 22.1 mm
- net Net-(J1-Pin_1): track 79.0 -> 95.7 mm
- net /celda_1/bus_pos: track 236.3 -> 247.4 mm
- net /celda_4/cell_neg: track 17.4 -> 26.3 mm
- net Net-(VCELL6-+): track 17.5 -> 11.2 mm
- net /celda_6/cell_neg: track 18.1 -> 23.8 mm
- net Net-(VCELL4-+): track 16.8 -> 11.2 mm
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Other:
- board outline added: 271.5 x 102.5 mm
