File: Prototipo/prototipo.kicad_pcb (KiCad board)
At the start: 2 copper layers, 184.9 x 180.4 mm, 148 parts, among them Q11_1 MMBT2222A, Q11_2 MMBT2907A, Q11_3 MMBT2222A, Q12_1 MMBT2222A, Q12_2 MMBT2907A, Q12_3 MMBT2222A, Q1_1 MMBT2222A, Q1_2 MMBFJ201, Q21_1 MMBT2222A, Q21_2 MMBT2907A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

Commit message: doy vuelta el inversor para no tener que hacer tantas vías
Parts:
- removed IN1: Conn_01x12_Pin, Connector_PinHeader_2.54mm:PinHeader_1x12_P2.54mm_Vertical
- added J1: Conn_02x12_Odd_Even, Connector_PinHeader_2.54mm:PinHeader_2x12_P2.54mm_Vertical, F.Cu at (20.6, 109.1)
- added J_B3: Conn_01x02_Pin, Connector_PinHeader_2.54mm:PinHeader_1x02_P2.54mm_Vertical, F.Cu at (72.7, 30.1)
- A1: moved to B.Cu
- moved TP_tierra1 417.9 mm to (-25.9, -56.4)
- moved TP_tierra3 417.9 mm to (-19.5, -63.6)
- moved TP_tierra4 417.9 mm to (-13.3, -53.3)
- moved TPgnd12 417.9 mm to (-24.9, -48.7)
- moved TPgnd22 417.9 mm to (-7.20, -59.5)
- moved TPgnd32 417.9 mm to (-17.4, -44.4)
- moved TPgnd21 365.5 mm to (89.9, 186.7)
- moved TPgnd31 364.7 mm to (144.7, 186.7)
- moved VCELL22 364.2 mm to (130.6, 107.5)
- moved Q32_1 364.2 mm to (161.2, 51.9)
- moved Rout32 364.2 mm to (148.3, 82.1)
- moved F3 364.2 mm to (159.1, 139.4)
- moved Q11_3 364.2 mm to (48.2, 183.7)
- moved Q12_1 364.2 mm to (72.7, 52.1)
- moved Q22_1 364.2 mm to (115.7, 51.9)
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Routing:
- net Vc_31: track 168.9 -> 262.0 mm, vias 2 -> 0
- net Vc_21: track 140.1 -> 204.2 mm, vias 2 -> 0
- net /celda_21/Vcontrol_neg: track 225.0 -> 168.2 mm
- net VCC: track 14.9 -> 66.5 mm, vias 0 -> 2
- net /celda_11/bus_neg: track 129.8 -> 164.2 mm
- net /celda_32/cell_neg: track 78.9 -> 54.9 mm
- net /celda_21/bus_pos: track 355.8 -> 334.0 mm
- net /celda_12/Vcontrol_neg: track 78.0 -> 57.5 mm, vias 0 -> 1
- net /celda_31/Vcontrol_neg: track 215.6 -> 199.9 mm
- net Vc_11: track 120.5 -> 134.8 mm, vias 2 -> 0
- net Vc3: track 115.8 -> 124.8 mm, vias 0 -> 1
- net /celda_22/Vcontrol_neg: track 109.5 -> 103.0 mm, vias 0 -> 1
- net Net-(J_B1-Pin_2): track 107.1 -> 100.7 mm
- net Vc2: track 63.7 -> 70.0 mm, vias 0 -> 1
- net /celda_31/bus_pos: track 212.1 -> 217.3 mm
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- added copper zone on B.Cu, net 0

Commit message: acomodo devuelta el inversor, y agrego conectores para medir con el micro
Parts:
- removed TP_tierra1, TP_tierra2, TP_tierra3, TP_tierra4: TestPoint, TestPoint:TestPoint_Bridge_Pitch2.54mm_Drill1.0mm
- added ?: , , F.Cu at (497.1, 203.2)
- added ?: , , F.Cu at (325.1, 29.8)
- added ?: , , F.Cu at (324.1, 202.1)
- added ?: , , F.Cu at (496.1, 28.3)
- added Celdas_bus1: Conn_01x02_Pin, Connector_PinHeader_2.54mm:PinHeader_1x02_P2.54mm_Vertical, F.Cu at (497.7, 116.3)
- added Celdas_inf1: Conn_01x03_Pin, Connector_PinHeader_2.54mm:PinHeader_1x03_P2.54mm_Vertical, F.Cu at (473.2, 203.4)
- added Celdas_sup1: Conn_01x03_Pin, Connector_PinHeader_2.54mm:PinHeader_1x03_P2.54mm_Vertical, F.Cu at (472.8, 30.1)
- A1: moved to F.Cu
- moved TPgnd32 492.6 mm to (454.1, 98.5)
- moved TPgnd22 452.9 mm to (425.9, 72.9)
- moved TPgnd12 424.5 mm to (384.8, 62.8)
- moved J_B3 309.8 mm to (382.4, 32.8)
- moved J_B2 309.6 mm to (459.5, 32.8)
- moved TPC11 309.6 mm to (347.2, 152.7)
- moved J_B1 309.4 mm to (412.1, 32.8)
- moved D2 309.3 mm to (396.8, 130.9)
- moved D21 309.3 mm to (392.3, 180.8)
- moved D22 309.3 mm to (415.7, 105.2)
- moved D31 309.3 mm to (446.2, 180.8)
- moved F12 309.3 mm to (380.9, 90.2)
- moved F2 309.3 mm to (414.6, 143.0)
- moved F21 309.3 mm to (414.6, 169.7)
- moved F31 309.3 mm to (468.4, 169.7)
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Connections:
- A1 pad 1: Vc_11 -> Vc_21
- A1 pad 2: /celda_11/Vcontrol_neg -> /celda_21/Vcontrol_neg
- A1 pad 3: Vc_21 -> Vc_11
- A1 pad 4: /celda_21/Vcontrol_neg -> /celda_11/Vcontrol_neg
- J1 pad 10: Vc3 -> Vc_11
- J1 pad 11: Vc_11 -> Vc_21
- J1 pad 12: Vc_11 -> Vc_21
- J1 pad 13: Vc_21 -> Vc_31
- J1 pad 14: Vc_21 -> Vc_31
- J1 pad 15: Vc_31 -> Vc_12
- J1 pad 16: Vc_31 -> Vc_12
- J1 pad 17: Vc_12 -> Vc_22
- J1 pad 18: Vc_12 -> Vc_22
- J1 pad 19: Vc_22 -> Vc_32
- J1 pad 20: Vc_22 -> Vc_32
- J1 pad 21: Vc_32 -> VCC
- J1 pad 22: Vc_32 -> VCC
- J1 pad 3: VCC -> Vc1
- J1 pad 4: VCC -> Vc1
- J1 pad 5: Vc1 -> Vc2
- J1 pad 6: Vc1 -> Vc2
- J1 pad 7: Vc2 -> Vc3
- J1 pad 8: Vc2 -> Vc3
- J1 pad 9: Vc3 -> Vc_11
Routing:
- net /celda_11/cell_neg: track 72.0 -> 181.0 mm
- net /celda_12/cell_neg: track 82.8 -> 168.0 mm, vias 0 -> 2
- net /celda_11/bus_pos: track 288.5 -> 370.7 mm
- net /celda_21/cell_neg: track 57.8 -> 114.3 mm
- net /celda_22/cell_neg: track 77.0 -> 119.8 mm, vias 0 -> 2
- net /celda_21/bus_pos: track 334.0 -> 373.1 mm
- net VCC: track 66.5 -> 35.2 mm, vias 2 -> 0
- net /celda_32/Vcontrol_neg: track 155.0 -> 128.4 mm, vias 1 -> 0
- net Vc_31: track 262.0 -> 288.0 mm, vias 0 -> 1
- net /celda_22/Vcontrol_neg: track 103.0 -> 91.2 mm, vias 1 -> 0
- net /celda_31/cell_neg: track 57.8 -> 67.6 mm
- net Vc_22: track 145.6 -> 154.5 mm, vias 1 -> 2
- net /celda_31/bus_pos: track 217.3 -> 225.5 mm
- net /celda_32/cell_neg: track 54.9 -> 63.1 mm
- net Vc_12: track 102.1 -> 109.9 mm, vias 1 -> 0
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Other:
- board size 184.9 x 180.4 mm -> 180.1 x 180.5 mm

Commit message: Sumo ultimos cambios hablados en reunion
agrega agujeros para tornillos, jumper para banco 1, INVERSOR CON ZOCALO, cambia el diametro de test points y vias, acomoda serigrafia, SIN WARNINGS
Parts:
- removed ? (x4): , 
- added H1: MountingHole, MountingHole:MountingHole_3.2mm_M3, F.Cu at (16.9, 206.8)
- added H2: MountingHole, MountingHole:MountingHole_3.2mm_M3, F.Cu at (192.8, 206.8)
- added H3: MountingHole, MountingHole:MountingHole_3.2mm_M3, F.Cu at (17.1, 31.8)
- added H4: MountingHole, MountingHole:MountingHole_3.2mm_M3, F.Cu at (192.8, 31.8)
- added J_B4: Conn_01x02_Pin, Connector_PinHeader_2.54mm:PinHeader_1x02_P2.54mm_Vertical, F.Cu at (86.4, 32.9)
- moved S3 307.2 mm to (144.5, 149.0)
- moved A1 307.1 mm to (29.0, 69.5)
- moved Celdas_bus1 307.1 mm to (190.6, 119.0)
- moved Celdas_inf1 307.1 mm to (166.1, 206.1)
- moved Celdas_sup1 307.1 mm to (165.6, 32.8)
- moved D1 307.1 mm to (35.8, 133.5)
- moved D11 307.1 mm to (31.3, 182.9)
- moved D12 307.1 mm to (66.7, 108.2)
- moved D2 307.1 mm to (89.7, 133.6)
- moved D21 307.1 mm to (85.2, 183.4)
- moved D22 307.1 mm to (108.6, 107.8)
- moved D3 307.1 mm to (143.5, 133.4)
- moved D31 307.1 mm to (139.1, 183.4)
- moved D32 307.1 mm to (154.0, 107.8)
- moved F1 307.1 mm to (53.6, 145.6)
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Connections:
- J1 pad 15: Vc_12 -> Vc_22
- J1 pad 16: Vc_12 -> Vc_22
- J1 pad 17: Vc_22 -> Vc_12
- J1 pad 18: Vc_22 -> Vc_12
Routing:
- net /celda_11/bus_pos: track 370.7 -> 445.9 mm
- net Vc_22: track 154.5 -> 173.8 mm, vias 2 -> 1
- net /celda_11/bus_neg: track 165.3 -> 172.8 mm
- net Vc_31: track 288.0 -> 281.2 mm, vias 1 -> 0
- net /celda_22/cell_neg: track 119.8 -> 114.2 mm
- net /celda_12/cell_neg: track 168.0 -> 162.7 mm
- net /celda_31/bus_pos: track 225.5 -> 220.7 mm
- net /celda_22/Vcontrol_neg: track 91.2 -> 87.0 mm, vias 0 -> 1
- net /celda_11/cell_neg: track 181.0 -> 177.4 mm
- net VCC: track 35.2 -> 38.2 mm
- net /celda_12/Vcontrol_neg: track 55.6 -> 53.4 mm
- net Net-(Q1_1-C): track 24.6 -> 22.6 mm
- net Net-(Q3_1-C): track 24.2 -> 22.2 mm
- net Net-(Q2_1-C): track 24.0 -> 22.0 mm
- net Net-(Q12_2-B): track 31.4 -> 29.5 mm
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Other:
- board size 180.1 x 180.5 mm -> 186 x 185 mm

Commit message: borrar mas textos innecesarios
Routing:
- net /celda_21/bus_pos: track 372.6 -> 375.2 mm
- net /celda_31/Vcontrol_neg: track 204.9 -> 206.3 mm

Commit message: Suma leds a kicad, falta rutear
Parts:
- added DLED1: LED, LED_THT:LED_D5.0mm, F.Cu at (-98.9, 157.8)
- added DLED11: LED, LED_THT:LED_D5.0mm, F.Cu at (45.9, 117.4)
- added DLED12: LED, LED_THT:LED_D5.0mm, F.Cu at (-113.5, 140.3)
- added DLED2: LED, LED_THT:LED_D5.0mm, F.Cu at (-81.4, 196.7)
- added DLED21: LED, LED_THT:LED_D5.0mm, F.Cu at (-98.9, 140.3)
- added DLED22: LED, LED_THT:LED_D5.0mm, F.Cu at (-128.1, 157.8)
- added DLED3: LED, LED_THT:LED_D5.0mm, F.Cu at (-113.5, 157.8)
- added DLED31: LED, LED_THT:LED_D5.0mm, F.Cu at (-109.8, 189.8)
- added DLED32: LED, LED_THT:LED_D5.0mm, F.Cu at (-128.1, 140.3)
- added QLED1: MMBT2222A, Package_TO_SOT_SMD:SOT-23-3, F.Cu at (31.4, 114.0)
- added QLED2: MMBT2222A, Package_TO_SOT_SMD:SOT-23-3, F.Cu at (-91.3, 173.9)
- added QLED21: MMBT2222A, Package_TO_SOT_SMD:SOT-23-3, F.Cu at (-91.3, 138.8)
- added QLED22: MMBT2222A, Package_TO_SOT_SMD:SOT-23-3, F.Cu at (-120.5, 156.3)
- added QLED3: MMBT2222A, Package_TO_SOT_SMD:SOT-23-3, F.Cu at (-105.9, 156.3)
- added QLED31: MMBT2222A, Package_TO_SOT_SMD:SOT-23-3, F.Cu at (-105.9, 173.9)
- added QLED32: MMBT2222A, Package_TO_SOT_SMD:SOT-23-3, F.Cu at (-120.5, 138.8)
- added QLED_11: MMBT2222A, Package_TO_SOT_SMD:SOT-23-3, F.Cu at (-120.5, 173.9)
- added QLED_12: MMBT2222A, Package_TO_SOT_SMD:SOT-23-3, F.Cu at (-105.9, 138.8)
- added RLED11_1: 20k, Resistor_THT:R_Axial_DIN0207_L6.3mm_D2.5mm_P7.62mm_Horizontal, F.Cu at (-129.0, 165.6)
- added RLED11_2: 1k, Resistor_THT:R_Axial_DIN0207_L6.3mm_D2.5mm_P7.62mm_Horizontal, F.Cu at (-129.0, 169.7)
- added RLED12_1: 20k, Resistor_THT:R_Axial_DIN0207_L6.3mm_D2.5mm_P7.62mm_Horizontal, F.Cu at (-114.4, 130.5)
- added RLED12_2: 1k, Resistor_THT:R_Axial_DIN0207_L6.3mm_D2.5mm_P7.62mm_Horizontal, F.Cu at (-114.4, 134.5)
- added RLED1_1: 20k, Resistor_THT:R_Axial_DIN0207_L6.3mm_D2.5mm_P7.62mm_Horizontal, F.Cu at (34.9, 114.0)
- added RLED1_2: 1K, Resistor_THT:R_Axial_DIN0207_L6.3mm_D2.5mm_P7.62mm_Horizontal, F.Cu at (34.9, 118.0)
- added RLED21_1: 20k, Resistor_THT:R_Axial_DIN0207_L6.3mm_D2.5mm_P7.62mm_Horizontal, F.Cu at (-99.7, 130.5)
- added RLED21_2: 1k, Resistor_THT:R_Axial_DIN0207_L6.3mm_D2.5mm_P7.62mm_Horizontal, F.Cu at (-99.7, 134.5)
- added RLED22_1: 20k, Resistor_THT:R_Axial_DIN0207_L6.3mm_D2.5mm_P7.62mm_Horizontal, F.Cu at (-129.0, 148.0)
- added RLED22_2: 1k, Resistor_THT:R_Axial_DIN0207_L6.3mm_D2.5mm_P7.62mm_Horizontal, F.Cu at (-129.0, 152.1)
- added RLED2_1: 20k, Resistor_THT:R_Axial_DIN0207_L6.3mm_D2.5mm_P7.62mm_Horizontal, F.Cu at (-99.7, 165.6)
- added RLED2_2: 1K, Resistor_THT:R_Axial_DIN0207_L6.3mm_D2.5mm_P7.62mm_Horizontal, F.Cu at (-99.7, 169.7)
- added RLED31_1: 20k, Resistor_THT:R_Axial_DIN0207_L6.3mm_D2.5mm_P7.62mm_Horizontal, F.Cu at (-114.4, 165.6)
- added RLED31_2: 1k, Resistor_THT:R_Axial_DIN0207_L6.3mm_D2.5mm_P7.62mm_Horizontal, F.Cu at (-114.4, 169.7)
- added RLED32_1: 20k, Resistor_THT:R_Axial_DIN0207_L6.3mm_D2.5mm_P7.62mm_Horizontal, F.Cu at (-129.0, 130.5)
- added RLED32_2: 1k, Resistor_THT:R_Axial_DIN0207_L6.3mm_D2.5mm_P7.62mm_Horizontal, F.Cu at (-129.0, 134.5)
- added RLED3_1: 20k, Resistor_THT:R_Axial_DIN0207_L6.3mm_D2.5mm_P7.62mm_Horizontal, F.Cu at (-114.4, 148.0)
- added RLED3_2: 1K, Resistor_THT:R_Axial_DIN0207_L6.3mm_D2.5mm_P7.62mm_Horizontal, F.Cu at (-114.4, 152.1)
Routing:
- net /celda_31/Vcontrol_neg: track 206.3 -> 207.8 mm
- net /celda_11/Vcontrol_neg: track 154.0 -> 153.5 mm
