File: Prototipo/celda.kicad_sch (KiCad schematic)
At the start: 22 parts, among them Q11_1 MMBT2222A, Q11_2 MMBT2907A, Q11_3 MMBT2222A

Commit message: se suman los leds al pcb
Parts:
- renumbered QLED_11 to QLED11
Connections:
- net bus_pos: no longer DLED11.2 (A)
- new net vcc: DLED11.2 (A)
Changed lines of the file:
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@@
-	)
-	(junction
-		(at 110.49 48.26)
-		(diameter 0)
-		(color 0 0 0 0)
 	)
 	(junction
@@
 			(width 0)
 			(type default)
-		)
-	)
-	(wire
-		(pts
-			(xy 110.49 48.26) (xy 69.85 48.26)
-		)
-		(stroke
-			(width 0.1524)
-			(type solid)
 		)
 	)
@@
 		(shape input)
 		(at 171.45 77.47 0)
+		(effects
+			(font
+				(size 1.27 1.27)
+			)
+			(justify left)
+		)
+	)
+	(hierarchical_label "vcc"
+		(shape input)
+		(at 69.85 48.26 90)
 		(effects
 			(font
@@
 		(on_board yes)
 		(dnp no)
-		(property "Reference" "QLED_11"
+		(property "Reference" "QLED11"
 			(at 69.215 72.39 0)
 			(effects
@@
 				)
 				(path "/c9225433-a7fd-41e8-8162-e91e829dcb79/6883bdf6-06e3-408b-a2b6-79a0e0cc9199"
-					(reference "QLED_11")
-					(unit 1)
-				)
+					(reference "QLED11")
+					(unit 1)
+				)
