File: Prototipo/PCB/prototipo.kicad_pcb (KiCad board)
At the start: 2 copper layers, 188.4 x 185 mm, 189 parts, among them J1 Conn_02x12_Odd_Even, Q11_1 MMBT2222A, Q11_2 MMBT2907A, Q11_3 MMBT2222A, Q12_1 MMBT2222A, Q12_2 MMBT2907A, Q12_3 MMBT2222A, Q1_1 MMBT2222A, Q1_2 MMBFJ201, Q21_1 MMBT2222A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

Commit message: Meto todo lo del prototipo en una carpeta
Routing:
- net Net-(VCELL22-+): track 33.8 -> 35.3 mm
Changed lines of the file:
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@@
 	)
 	(segment
-		(start 816.913001 101.47)
-		(end 816.913001 106.68)
+		(start 816.4 101.983001)
+		(end 816.4 108)
+		(width 1.2)
+		(layer "B.Cu")
+		(net 86)
+	)
+	(segment
+		(start 816.4 108)
+		(end 835.27 126.87)
 		(width 1.2)
 		(layer "B.Cu")
@@
 	)
 	(segment
-		(start 816.913001 106.68)
+		(start 835.27 126.87)
 		(end 837.103001 126.87)
 		(width 1.2)
@@
 	)
 	(segment
+		(start 816.913001 101.47)
+		(end 816.4 101.983001)
+		(width 1.2)
+		(layer "B.Cu")
+		(net 86)
+	)
+	(segment
 		(start 866.0545 167.77)
 		(end 877.85 155.9745)
@@
 			)
 		)
+	)
+	(zone
+		(net 86)
+		(net_name "Net-(VCELL22-+)")
+		(layer "B.Cu")
+		(name "$teardrop_padvia$")
+		(hatch none 0.1)
+		(priority 30000)
+		(attr
+			(teardrop
+				(type padvia)
+			)
+		)
+		(connect_pads yes
+			(clearance 0)
+		)
+		(min_thickness 0.0254)
+		(filled_areas_thickness no)
+		(fill yes
+			(thermal_gap 0.5)
+			(thermal_bridge_width 0.5)
+			(island_removal_mode 1)
+			(island_area_min 10)
+		)
+		(polygon
+			(pts
+				(xy 817 102.866631) (xy 817.004889 102.746102) (xy 817.019109 102.645439) (xy 817.039904 102.56733)
+				(xy 817.067536 102.500568) (xy 817.1433 102.388038) (xy 817.269398 102.263047) (xy 817.415764 102.120309)
+				(xy 817.495469 102.027829) (xy 817.578177 101.914456) (xy 816.913001 101.469) (xy 816.128373 101.313928)
+				(xy 816.036741 101.69141) (xy 815.948444 101.960904) (xy 815.88952 102.13704) (xy 815.842463 102.324306)
+				(xy 815.811285 102.556303) (xy 815.8 102.866631)
+			)
+		)

Commit message: Sube archivos de fabricación
Parts:
- moved Celdas_inf1 660.0 mm to (211.0, 248.0)
- moved Celdas_sup1 660.0 mm to (210.6, 74.7)
- moved D1 660.0 mm to (80.8, 175.4)
- moved D11 660.0 mm to (76.3, 224.8)
- moved D3 660.0 mm to (188.5, 175.3)
- moved F1 660.0 mm to (98.5, 187.6)
- moved F11 660.0 mm to (98.5, 214.3)
- moved F12 660.0 mm to (118.8, 134.8)
- moved F3 660.0 mm to (206.2, 187.4)
- moved J1 660.0 mm to (62.3, 191.5)
- moved J_B1 660.0 mm to (150.0, 77.3)
- moved J_B2 660.0 mm to (198.7, 77.2)
- moved J_B3 660.0 mm to (120.9, 74.8)
- moved J_B4 660.0 mm to (131.4, 74.8)
- moved OUT1 660.0 mm to (104.2, 75.7)
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Routing:
- net /celda_11/bus_neg: track 164.1 -> 166.0 mm
