File: hardware/Circuito Final/Switch banco - Torre/Switch banco - Torre.kicad_sch (KiCad schematic)
At the start: 69 parts, among them J1 Conn_01x07, J2 Conn_02x07_Odd_Even, J3 Conn_01x07, Q1 MMBFJ112, Q1_1 MMBT2222A, Q3 MMBT2222A, U1 74HC595, U2 74HC4051

Commit message: prueba del mux, y bitacora del dia
Other:
- moved on the sheet: J2
Changed lines of the file:
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@@
 	(wire
 		(pts
-			(xy 144.78 144.78) (xy 148.59 144.78)
+			(xy 147.32 153.67) (xy 151.13 153.67)
 		)
 		(stroke
@@
 	(wire
 		(pts
+			(xy 149.86 151.13) (xy 151.13 151.13)
+		)
+		(stroke
+			(width 0)
+			(type default)
+		)
+	)
+	(wire
+		(pts
 			(xy 49.53 95.25) (xy 48.26 95.25)
 		)
@@
 	(wire
 		(pts
-			(xy 132.08 142.24) (xy 148.59 142.24)
-		)
-		(stroke
-			(width 0)
-			(type default)
-		)
-	)
-	(wire
-		(pts
 			(xy 80.01 31.75) (xy 80.01 20.32)
 		)
@@
 	)
 	(label "DATA"
-		(at 161.29 147.32 0)
+		(at 163.83 156.21 0)
 		(effects
 			(font
@@
 	)
 	(label "salida_adc"
-		(at 161.29 134.62 0)
+		(at 163.83 143.51 0)
 		(effects
 			(font
@@
 	)
 	(label "bus_pos"
-		(at 161.29 137.16 0)
+		(at 163.83 146.05 0)
 		(effects
 			(font
@@
 	)
 	(label "bus_neg"
-		(at 161.29 139.7 0)
+		(at 163.83 148.59 0)
 		(effects
 			(font
@@
 	)
 	(label "clock"
-		(at 144.78 144.78 180)
+		(at 147.32 153.67 180)
 		(effects
 			(font
@@
 	)
 	(label "Bit_0"
-		(at 161.29 132.08 0)
+		(at 163.83 140.97 0)
 		(effects
 			(font
@@
 	)
 	(label "latch"
-		(at 161.29 144.78 0)
+		(at 163.83 153.67 0)
 		(effects
 			(font
@@
 	)
 	(label "Bit_1"
-		(at 148.59 132.08 180)
+		(at 151.13 140.97 180)
 		(effects
 			(font
@@
 	)
 	(label "Bit_2"
-		(at 148.59 134.62 180)
+		(at 151.13 143.51 180)
 		(effects
 			(font
@@
 	)
 	(label "Vcc"
-		(at 148.59 147.32 180)
+		(at 151.13 156.21 180)
 		(effects
 			(font
@@
 	)
 	(label "bus_neg"
-		(at 148.59 139.7 180)
+		(at 151.13 148.59 180)
 		(effects
 			(font
@@
 	)
 	(label "bus_pos"
-		(at 148.59 137.16 180)
+		(at 151.13 146.05 180)
 		(effects
 			(font
@@
 	(symbol
 		(lib_id "power:GND")
-		(at 132.08 142.24 270)
+		(at 149.86 151.13 270)
 		(unit 1)
 		(body_style 1)
@@
 		(fields_autoplaced yes)
 		(property "Reference" "#PWR033"
-			(at 125.73 142.24 0)
+			(at 143.51 151.13 0)
 			(hide yes)
 			(show_name no)
@@
 		)
 		(property "Value" "GND"
-			(at 128.27 142.2399 90)
+			(at 146.05 151.1299 90)
 			(show_name no)
 			(do_not_autoplace no)
@@
 		)
 		(property "Footprint" ""
-			(at 132.08 142.24 0)
+			(at 149.86 151.13 0)
 			(hide yes)
 			(show_name no)
@@
 		)
 		(property "Datasheet" ""
-			(at 132.08 142.24 0)
+			(at 149.86 151.13 0)
 			(hide yes)
 			(show_name no)
@@
 		)
 		(property "Description" "Power symbol creates a global label with name \"GND\" , ground"
-			(at 132.08 142.24 0)
+			(at 149.86 151.13 0)
 			(hide yes)
 			(show_name no)
@@
 	(symbol
 		(lib_id "Connector_Generic:Conn_02x07_Odd_Even")
-		(at 153.67 139.7 0)
+		(at 156.21 148.59 0)
 		(unit 1)
 		(body_style 1)
@@
 		(fields_autoplaced yes)
 		(property "Reference" "J2"
-			(at 154.94 125.73 0)
+			(at 157.48 134.62 0)
 			(show_name no)
 			(do_not_autoplace no)
@@
 		)
 		(property "Value" "Conn_02x07_Odd_Even"
-			(at 154.94 128.27 0)
+			(at 157.48 137.16 0)
 			(show_name no)
 			(do_not_autoplace no)
@@
 		)
 		(property "Footprint" "Connector_IDC:IDC-Header_2x07_P2.54mm_Horizontal"
-			(at 153.67 139.7 0)
+			(at 156.21 148.59 0)
 			(hide yes)
 			(show_name no)
@@
 		)
 		(property "Datasheet" ""
-			(at 153.67 139.7 0)
+			(at 156.21 148.59 0)
 			(hide yes)
 			(show_name no)
@@
 		)
 		(property "Description" "Generic connector, double row, 02x07, odd/even pin numbering scheme (row 1 odd numbers, row 2 even numbers), script generated (kicad-library-utils/schlib/autogen/connector/)"
-			(at 153.67 139.7 0)
+			(at 156.21 148.59 0)
 			(hide yes)
 			(show_name no)
@@
 	(symbol
 		(lib_id "power:GND")
-		(at 161.29 142.24 90)
+		(at 163.83 151.13 90)
 		(unit 1)
 		(body_style 1)
@@
 		(fields_autoplaced yes)
 		(property "Reference" "#PWR018"
-			(at 167.64 142.24 0)
+			(at 170.18 151.13 0)
 			(hide yes)
 			(show_name no)
@@
 		)
 		(property "Value" "GND"
-			(at 165.1 142.2399 90)
+			(at 167.64 151.1299 90)
 			(show_name no)
 			(do_not_autoplace no)
@@
 		)
 		(property "Footprint" ""
-			(at 161.29 142.24 0)
+			(at 163.83 151.13 0)
 			(hide yes)
 			(show_name no)
@@
 		)
 		(property "Datasheet" ""
-			(at 161.29 142.24 0)
+			(at 163.83 151.13 0)
 			(hide yes)
 			(show_name no)
@@
 		)
 		(property "Description" "Power symbol creates a global label with name \"GND\" , ground"
-			(at 161.29 142.24 0)
+			(at 163.83 151.13 0)
 			(hide yes)
 			(show_name no)
