File: hardware/Circuito Final/Switch banco - Torre/Switch banco - Torre.kicad_sch (KiCad schematic)
At the start: 69 parts, among them J1 Conn_01x07, J2 Conn_02x07_Odd_Even, J3 Conn_01x07, Q1 MMBFJ112, Q1_1 MMBT2222A, Q3 MMBT2222A, U1 74HC595, U2 74HC4051

Commit message: version 2.2 Banco
Parts:
- removed Rp1, Rp2, Rp3, Rp4, Rp5, Rp6, Rp7, Rp8: 10k, Resistor_SMD:R_1206_3216Metric_Pad1.30x1.75mm_HandSolder, symbol Device:R
