File: hardware/Circuito Final/Circuito externo/Circuito Final - Circuito externo.kicad_pcb (KiCad board)
At the start: 2 copper layers, 121 x 100.5 mm, 34 parts, among them J1 Conn_02x19_Odd_Even, J2 Conn_02x19_Odd_Even, J3 Conn_01x02, J4 Conn_01x02, SW1 SW_SPDT, SW2 SW_DIP_x04, U1 Opamp_Quad, U2 ICL7660

Commit message: sube nuevas conexiones, falta conectar los buses a los conectores
Parts:
- added SW3: SW_DIP_x04, Button_Switch_THT:SW_DIP_SPSTx04_Slide_9.78x12.34mm_W7.62mm_P2.54mm, B.Cu at (441.9, 74.6)
- added SW4: SW_DIP_x01, Button_Switch_THT:SW_DIP_SPSTx01_Slide_6.7x4.1mm_W7.62mm_P2.54mm_LowProfile, B.Cu at (479.3, 65.1)
- added SW5: SW_DIP_x01, Button_Switch_THT:SW_DIP_SPSTx01_Slide_6.7x4.1mm_W7.62mm_P2.54mm_LowProfile, B.Cu at (449.8, 65.1)
- added SW6: SW_DIP_x01, Button_Switch_THT:SW_DIP_SPSTx01_Slide_6.7x4.1mm_W7.62mm_P2.54mm_LowProfile, B.Cu at (420.2, 65.1)
- added TP1: TestPoint, TestPoint:TestPoint_Keystone_5005-5009_Compact, F.Cu at (549.8, -72.2)
- added TP2: TestPoint, TestPoint:TestPoint_Keystone_5005-5009_Compact, F.Cu at (549.8, -67.1)
- moved SW1 450.4 mm to (577.7, 18.2)
- moved C1 435.9 mm to (526.2, -1.65), turned to 180 degrees
- moved Bornera1 425.9 mm to (523.8, -7.53)
- moved G*** 375.0 mm to (553.5, -118.3)
- moved Jsalida_3 370.9 mm to (438.1, 54.9), turned to 90 degrees
- moved SW2 365.7 mm to (446.0, 37.0), turned to 90 degrees
- moved R12 365.6 mm to (461.7, 11.1)
- moved R22 356.9 mm to (456.5, 35.3), turned to -90 degrees
- moved R11 351.5 mm to (452.8, 35.4), turned to 90 degrees
- moved Rx2 351.0 mm to (457.3, 5.97)
- moved Rf2 350.7 mm to (448.1, 2.42), turned to 90 degrees
- moved R21 347.2 mm to (447.1, 34.2)
- moved J1 346.7 mm to (473.2, -29.1)
- moved J2 346.7 mm to (412.3, -29.1)
- moved J3 346.7 mm to (475.8, -57.1)
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Connections:
- J1 pad 1: /clk_latch -> /latch
- J1 pad 2: /clk_shift -> /clock
- Jsalida_1 pad 11: /clk_latch -> /clock
- Jsalida_1 pad 12: /reset -> /latch
- Jsalida_1 pad 9: /clk_shift -> GND
- Jsalida_2 pad 11: /clk_latch -> /clock
- Jsalida_2 pad 12: /reset -> /latch
- Jsalida_2 pad 7: /bus_pos_1 -> /bus_neg_2
- Jsalida_2 pad 8: /bus_pos_1 -> /bus_neg_2
- Jsalida_2 pad 9: /clk_shift -> GND
- Jsalida_3 pad 11: /clk_latch -> /clock
- Jsalida_3 pad 12: /reset -> /latch
- Jsalida_3 pad 7: /bus_pos_2 -> /bus_neg_3
- Jsalida_3 pad 8: /bus_pos_2 -> /bus_neg_3
- Jsalida_3 pad 9: /clk_shift -> GND
- Jsalida_4 pad 11: /clk_latch -> /clock
- Jsalida_4 pad 12: /reset -> /latch
- Jsalida_4 pad 7: /bus_pos_3 -> /bus_neg_4
- Jsalida_4 pad 8: /bus_pos_3 -> /bus_neg_4
- Jsalida_4 pad 9: /clk_shift -> GND
- R31 pad 1: /bus_pos_3 -> /bus_pos_4
- R32 pad 2: /bus_pos_2 -> /bus_pos_3
- R41 pad 1: /bus_pos_4 -> /bus_pos_3
- R42 pad 2: /bus_pos_3 -> /bus_pos_2
- Rf3 pad 2: /banco3_med -> /banco4_med
- Rf4 pad 2: /banco4_med -> /banco3_med
- U1 pad 14: /banco4_med -> /banco3_med
- U1 pad 8: /banco3_med -> /banco4_med
Routing:
- net /Bit_2: track 0.00 -> 249.6 mm, vias 0 -> 6
- net /latch: track 0.00 -> 205.0 mm, vias 0 -> 2
- net /Bit_0: track 0.00 -> 197.7 mm, vias 0 -> 7
- net /clock: track 0.00 -> 197.1 mm, vias 0 -> 6
- net /Vcc_out: track 0.00 -> 150.4 mm
- net /Bit_1: track 0.00 -> 136.9 mm, vias 0 -> 4
- net /Data_3: track 0.00 -> 91.5 mm, vias 0 -> 1
- net /Data_2: track 0.00 -> 79.5 mm, vias 0 -> 2
- net /salida_adc_4: track 0.00 -> 79.4 mm, vias 0 -> 2
- net /Data_4: track 0.00 -> 78.9 mm
- net /bus_pos_1: track 0.00 -> 76.7 mm
- net /Data_1: track 0.00 -> 76.5 mm, vias 0 -> 1
- net /bus_neg_3: track 0.00 -> 68.0 mm
- net /bus_neg_2: track 0.00 -> 67.3 mm
- net /bus_pos_3: track 0.00 -> 66.0 mm
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Other:
- board outline removed

Commit message: sube mediciones de switching
Parts:
- moved C1 105.4 mm to (440.8, -63.5)
- moved Bornera1 105.2 mm to (438.5, -69.0)
- moved TP1 94.9 mm to (455.0, -74.0)
- moved TP2 94.9 mm to (455.0, -69.0)
- moved SW1 85.7 mm to (492.8, 6.80), turned to -90 degrees
Changed lines of the file:
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@@
 	(footprint "Capacitor_SMD:C_1206_3216Metric_Pad1.33x1.80mm_HandSolder"
 		(layer "F.Cu")
-		(at 526.1625 -1.65 180)
+		(at 440.8125 -63.475 180)
 		(descr "Capacitor SMD 1206 (3216 Metric), square (rectangular) end terminal, IPC-7351 nominal with elongated pad for handsoldering. (Body size source: IPC-SM-782 page 76, https://www.pcb-3d.com/wordpress/wp-content/uploads/ipc-sm-782a_amendment_1_and_2.pdf)")
 		(tags "capacitor handsolder")
@@
 	(footprint "TestPoint:TestPoint_Keystone_5005-5009_Compact"
 		(layer "F.Cu")
-		(at 549.834607 -72.189606)
+		(at 454.975 -74.05)
 		(descr "Keystone THM Compact Test Point 5005-5009, http://www.keyelco.com/product-pdf.cfm?p=1314")
 		(tags "Through Hole Mount Test Points")
@@
 	(footprint "TestPoint:TestPoint_Keystone_5005-5009_Compact"
 		(layer "F.Cu")
-		(at 549.834607 -67.139606)
+		(at 454.975 -69)
 		(descr "Keystone THM Compact Test Point 5005-5009, http://www.keyelco.com/product-pdf.cfm?p=1314")
 		(tags "Through Hole Mount Test Points")
@@
 	(footprint "Huellas:TerminalBlock_bornier-2_P5.08mm"
 		(layer "B.Cu")
-		(at 523.825 -7.525)
+		(at 438.52 -69.025)
 		(descr "simple 2-pin terminal block, pitch 5.08mm, revamped version of bornier2")
 		(tags "terminal block bornier2")
@@
 	(footprint "Button_Switch_THT:SW_Slide_SPDT_Straight_CK_OS102011MS2Q"
 		(layer "B.Cu")
-		(at 577.675 18.175 180)
+		(at 492.775 6.8 -90)
 		(descr "CuK miniature slide switch, OS series, SPDT, https://www.ckswitches.com/media/1428/os.pdf")
 		(tags "switch SPDT")
 		(property "Reference" "SW1"
-			(at 3.99 2.99 0)
+			(at 3.99 2.99 90)
 			(layer "B.SilkS")
 			(effects
@@
 		)
 		(property "Value" "SW_SPDT"
-			(at 2 -3 0)
+			(at 2 -3 90)
 			(layer "B.Fab")
 			(effects
@@
 		)
 		(property "Datasheet" ""
-			(at 0 0 0)
+			(at 0 0 90)
 			(unlocked yes)
 			(layer "B.Fab")
@@
 		)
 		(property "Description" "Switch, single pole double throw"
-			(at 0 0 0)
+			(at 0 0 90)
 			(unlocked yes)
 			(layer "B.Fab")
@@
 		(duplicate_pad_numbers_are_jumpers no)
 		(fp_line
-			(start 6.41 2.26)
-			(end 6.41 1.95)
+			(start -0.5 2.96)
+			(end 0 2.46)
 			(stroke
 				(width 0.12)
@@
 		)
 		(fp_line
-			(start 6.41 -2.26)
-			(end 6.41 -1.95)
+			(start 0.5 2.96)
+			(end -0.5 2.96)
 			(stroke
 				(width 0.12)
@@
 		)
 		(fp_line
-			(start 6.41 -2.26)
-			(end -2.41 -2.26)
+			(start 0 2.46)
+			(end 0.5 2.96)
 			(stroke
 				(width 0.12)
@@
 		)
 		(fp_line
-			(start 0.5 2.96)
-			(end -0.5 2.96)
+			(start -2.41 2.26)
+			(end 6.41 2.26)
 			(stroke
 				(width 0.12)
@@
 		)
 		(fp_line
-			(start 0 2.46)
-			(end 0.5 2.96)
+			(start 6.41 2.26)
+			(end 6.41 1.95)
 			(stroke
 				(width 0.12)
@@
 		)
 		(fp_line
-			(start -0.5 2.96)
-			(end 0 2.46)
+			(start -2.41 1.95)
+			(end -2.41 2.26)
 			(stroke
 				(width 0.12)
@@
 		)
 		(fp_line
-			(start -2.41 2.26)
-			(end 6.41 2.26)
+			(start -2.41 -2.26)
+			(end -2.41 -1.95)
 			(stroke
 				(width 0.12)
@@
 		)
 		(fp_line
-			(start -2.41 1.95)
-			(end -2.41 2.26)
+			(start 6.41 -2.26)
+			(end 6.41 -1.95)
 			(stroke
 				(width 0.12)
@@
 		)
 		(fp_line
-			(start -2.41 -2.26)
-			(end -2.41 -1.95)
+			(start 6.41 -2.26)
+			(end -2.41 -2.26)
 			(stroke
 				(width 0.12)
@@
 		)
 		(fp_line
-			(start 7.45 2.4)
-			(end 7.45 -2.4)
+			(start -3.45 2.4)
+			(end 7.45 2.4)
 			(stroke
 				(width 0.05)
@@
 		)
 		(fp_line
-			(start 7.45 -2.4)
-			(end -3.45 -2.4)
+			(start 7.45 2.4)
+			(end 7.45 -2.4)
 			(stroke
 				(width 0.05)
@@
 		)
 		(fp_line
-			(start -3.45 2.4)
-			(end 7.45 2.4)
+			(start -3.45 -2.4)
+			(end -3.45 2.4)
 			(stroke
 				(width 0.05)
@@
 		)
 		(fp_line
-			(start -3.45 -2.4)
-			(end -3.45 2.4)
+			(start 7.45 -2.4)
+			(end -3.45 -2.4)
 			(stroke
 				(width 0.05)
@@
 		)
 		(fp_line
-			(start 6.3 2.15)
-			(end 6.3 -2.15)
+			(start -2.3 2.15)
+			(end -0.5 2.15)
 			(stroke
 				(width 0.1)
@@
 		)
 		(fp_line
-			(start 6.3 -2.15)
-			(end -2.3 -2.15)
+			(start -0.5 2.15)
+			(end 0 1.65)
 			(stroke
 				(width 0.1)
@@
 		)
 		(fp_line
-			(start 4 1)
-			(end 4 -1)
+			(start 0.5 2.15)
+			(end 6.3 2.15)
 			(stroke
 				(width 0.1)
@@
 		)
 		(fp_line
-			(start 2 1)
-			(end 2 -1)
+			(start 6.3 2.15)
+			(end 6.3 -2.15)
 			(stroke
 				(width 0.1)
@@
 		)
 		(fp_line
-			(start 1.34 1)
-			(end 1.34 -1)
+			(start 0 1.65)
+			(end 0.5 2.15)
 			(stroke
 				(width 0.1)
@@
 		)
 		(fp_line
-			(start 0.66 1)
-			(end 0.66 -1)
+			(start 0 1)
+			(end 4 1)
 			(stroke
 				(width 0.1)
@@
 		)
 		(fp_line
-			(start 0.5 2.15)
-			(end 6.3 2.15)
+			(start 0 1)
+			(end 0 -1)
 			(stroke
 				(width 0.1)
@@
 		)
 		(fp_line
-			(start 0 1.65)
-			(end 0.5 2.15)
+			(start 0.66 1)
+			(end 0.66 -1)
 			(stroke
 				(width 0.1)
@@
 		)
 		(fp_line
-			(start 0 1)
-			(end 4 1)
+			(start 1.34 1)
+			(end 1.34 -1)
 			(stroke
 				(width 0.1)
@@
 		)
 		(fp_line
-			(start 0 1)
-			(end 0 -1)
+			(start 2 1)
+			(end 2 -1)
 			(stroke
 				(width 0.1)
@@
 		)
 		(fp_line
-			(start 0 -1)
+			(start 4 1)
 			(end 4 -1)
 			(stroke
@@
 		)
 		(fp_line
-			(start -0.5 2.15)
-			(end 0 1.65)
+			(start 0 -1)
+			(end 4 -1)
 			(stroke
 				(width 0.1)
@@
 		)
 		(fp_line
-			(start -2.3 2.15)
-			(end -0.5 2.15)
+			(start -2.3 -2.15)
+			(end -2.3 2.15)
 			(stroke
 				(width 0.1)
@@
 		)
 		(fp_line
-			(start -2.3 -2.15)
-			(end -2.3 2.15)
+			(start 6.3 -2.15)
+			(end -2.3 -2.15)
 			(stroke
 				(width 0.1)
@@
 		)
 		(fp_text user "${REFERENCE}"
-			(at 3.99 2.99 0)
+			(at 3.99 2.99 90)
 			(layer "B.Fab")
 			(effects
@@
 		)
 		(pad "" thru_hole oval
-			(at -2.1 0 180)
+			(at -2.1 0 270)
 			(size 2.2 3.5)
 			(drill 1.5)
@@
 		)
 		(pad "" thru_hole oval
-			(at 6.1 0 180)
+			(at 6.1 0 270)
 			(size 2.2 3.5)
 			(drill 1.5)
@@
 		)
 		(pad "1" thru_hole rect
-			(at 0 0 180)
+			(at 0 0 270)
 			(size 1.5 2.5)
 			(drill 0.8)
@@
 		)
 		(pad "2" thru_hole oval
-			(at 2 0 180)
+			(at 2 0 270)
 			(size 1.5 2.5)
 			(drill 0.8)
@@
 		)
 		(pad "3" thru_hole oval
-			(at 4 0 180)
+			(at 4 0 270)
 			(size 1.5 2.5)
 			(drill 0.8)
@@
 	)
 	(segment
-		(start 523.825 -2.425)
-		(end 524.6 -1.65)
+		(start 438.475 -64.25)
+		(end 439.25 -63.475)
 		(width 0.6)
 		(layer "F.Cu")
@@
 	)
 	(segment
-		(start 523.825 -7.525)
-		(end 523.825 -2.425)
+		(start 438.475 -69.35)
+		(end 438.475 -64.25)
 		(width 0.6)
 		(layer "F.Cu")
@@
 	)
 	(segment
-		(start 529.175 -3.1)
-		(end 529.175 -7.255)
+		(start 443.825 -64.925)
+		(end 443.825 -69.08)
 		(width 0.6)
 		(layer "F.Cu")
@@
 	)
 	(segment
-		(start 527.725 -1.65)
-		(end 529.175 -3.1)
+		(start 442.375 -63.475)
+		(end 443.825 -64.925)
 		(width 0.6)
 		(layer "F.Cu")
@@
 	)
 	(segment
-		(start 452.9 33.735)
-		(end 452.9 17.175)
+		(start 451.775 11.025)
+		(end 450.225 9.475)
 		(width 0.6)
 		(layer "F.Cu")
@@
 	)
 	(segment
-		(start 450.225 14.5)
-		(end 450.225 9.475)
+		(start 452.9 17.175)
+		(end 451.775 16.05)
 		(width 0.6)
 		(layer "F.Cu")
@@
 	)
 	(segment
-		(start 452.9 17.175)
-		(end 450.225 14.5)
+		(start 452.9 33.735)
+		(end 452.9 17.175)
+		(width 0.6)
+		(layer "F.Cu")
+		(net "Net-(U1A-+)")
+	)
+	(segment
+		(start 451.775 16.05)
+		(end 451.775 11.025)
 		(width 0.6)
 		(layer "F.Cu")
@@
 		(polygon
 			(pts
-				(xy 521.655 -9.525) (xy 530.905 -9.525) (xy 530.905 -5.525) (xy 521.655 -5.525)
+				(xy 436.275 -70.95) (xy 445.525 -70.95) (xy 445.525 -66.95) (xy 436.275 -66.95)
 			)
 		)
@@
 		(polygon
 			(pts
-				(xy 569.95 16.005) (xy 581.45 16.005) (xy 581.45 20.505) (xy 569.95 20.505)
+				(xy 490.605 14.525) (xy 490.605 3.025) (xy 495.105 3.025) (xy 495.105 14.525)
 			)
 		)
@@
 		)
 	)
+	(group ""
+		(members "014050a0-4b21-43a9-a53f-65e73f812678" "02401ab7-4976-414c-9f54-12b1a21c1545")
+	)
 	(embedded_fonts no)

Commit message: sube mediciones y comienza devuelta el conexionado del pcb
Parts:
- added U3: INA180A1, Package_TO_SOT_SMD:SOT-23-5, F.Cu at (511.0, 86.3)
- SW2, SW3: footprint Button_Switch_THT:SW_DIP_SPSTx04_Slide_9.78x12.34mm_W7.62mm_P2.54mm -> Button_Switch_THT:SW_DIP_SPSTx04_Slide_6.7x11.72mm_W7.62mm_P2.54mm_LowProfile
- SW4, SW5, SW6: footprint Button_Switch_THT:SW_DIP_SPSTx01_Slide_6.7x4.1mm_W7.62mm_P2.54mm_LowProfile -> Button_Switch_THT:SW_DIP_SPSTx01_Slide_9.78x4.72mm_W7.62mm_P2.54mm
- moved J2 216.1 mm to (572.6, 115.8)
- moved J3 216.1 mm to (636.1, 87.8)
- moved J4 216.1 mm to (572.6, 87.8)
- moved J1 216.1 mm to (633.6, 115.8)
- moved STM32 216.1 mm to (604.4, 125.0)
- moved Bornera1 162.8 mm to (576.1, 18.0)
- moved C1 162.8 mm to (578.4, 23.6)
- moved TP1 162.8 mm to (592.5, 13.0)
- moved TP2 162.8 mm to (592.5, 18.0)
- moved Rf3 144.4 mm to (478.0, 141.4), turned to -90 degrees
- moved Rf2 141.2 mm to (464.6, 142.7), turned to -90 degrees
- moved Rx3 139.3 mm to (483.2, 136.8), turned to 0 degrees
- moved Rx2 133.2 mm to (455.5, 139.1), turned to 180 degrees
- moved U1 133.1 mm to (471.5, 137.4), turned to 0 degrees
- moved Rx1 127.0 mm to (461.2, 135.9), turned to 180 degrees
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Routing:
- net /Bit_2: track 249.6 -> 0.00 mm, vias 6 -> 0
- net /latch: track 205.0 -> 0.00 mm, vias 2 -> 0
- net /Bit_0: track 197.7 -> 0.00 mm, vias 7 -> 0
- net /clock: track 197.1 -> 0.00 mm, vias 6 -> 0
- net /Bit_1: track 136.9 -> 0.00 mm, vias 4 -> 0
- net /Vcc_out: track 150.4 -> 20.9 mm
- net /Data_3: track 91.5 -> 0.00 mm, vias 1 -> 0
- net /Data_2: track 79.5 -> 0.00 mm, vias 2 -> 0
- net /salida_adc_4: track 79.4 -> 0.00 mm, vias 2 -> 0
- net /Data_4: track 78.9 -> 0.00 mm
- net /Data_1: track 76.5 -> 0.00 mm, vias 1 -> 0
- net /salida_adc_1: track 63.7 -> 0.00 mm
- net /salida_adc_3: track 58.0 -> 0.00 mm, vias 2 -> 0
- net /bus_pos_1: track 76.7 -> 20.1 mm
- net /salida_adc_2: track 48.5 -> 0.00 mm, vias 2 -> 0
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
Commit message: clasifica los bloques en el esquematico de kicad
Parts:
- added Bornera2: Conn_01x02_Socket, Huellas:TerminalBlock_bornier-2_P5.08mm, F.Cu at (364.2, 112.5)
- added C4: 100n, Capacitor_SMD:C_1206_3216Metric_Pad1.33x1.80mm_HandSolder, F.Cu at (414.4, 88.1)
- added Q1: FDMS6681Z, Huellas:FDMS6681Z, F.Cu at (403.5, 127.9)
- added Q2: FDMS6681Z, Huellas:FDMS6681Z, F.Cu at (403.5, 118.7)
- added Q3: MMBT2222A, Package_TO_SOT_SMD:SOT-23, F.Cu at (406.8, 138.8)
- added R1: 22k, Resistor_SMD:R_1206_3216Metric_Pad1.30x1.75mm_HandSolder, F.Cu at (407.6, 143.5)
- added R2: 1m, Resistor_SMD:R_2512_6332Metric_Pad1.40x3.35mm_HandSolder, F.Cu at (404.7, 88.1)
- added R3: 22k, Resistor_SMD:R_1206_3216Metric_Pad1.30x1.75mm_HandSolder, F.Cu at (405.1, 134.6)
- added R4: 1k, Resistor_SMD:R_1206_3216Metric_Pad1.30x1.75mm_HandSolder, F.Cu at (363.9, 118.7)
- added R5: 10k, Resistor_SMD:R_1206_3216Metric_Pad1.30x1.75mm_HandSolder, F.Cu at (363.9, 122.0)
- moved SW1 223.4 mm to (402.3, 108.4), turned to 90 degrees
- moved TP1 215.6 mm to (394.2, 97.6), turned to 180 degrees
- moved TP2 207.5 mm to (394.2, 78.9), turned to 180 degrees
- moved Bornera1 194.1 mm to (394.2, 85.7), turned to -90 degrees
- moved C1 189.3 mm to (400.4, 88.0), turned to 90 degrees
- moved J2 158.2 mm to (414.6, 107.6)
- moved J3 158.2 mm to (478.1, 79.6)
- moved J4 158.2 mm to (414.6, 79.6)
- moved J1 158.2 mm to (475.6, 107.6)
- moved STM32 158.2 mm to (446.4, 116.7)
- moved U3 101.3 mm to (409.7, 88.2), turned to -90 degrees
- moved SW2 71.7 mm to (443.1, 40.4)
- moved U1 59.0 mm to (443.8, 85.2), turned to 90 degrees
- moved R32 51.2 mm to (454.1, 77.8)
- moved R31 50.3 mm to (443.8, 77.9)
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Connections:
- Bornera1 pad 1: /bus_neg_1 -> /bus_neg_salida
- Bornera1 pad 2: /bus_pos_salida -> /shunt
- C1 pad 1: /bus_pos_salida -> /shunt
- C1 pad 2: /bus_neg_1 -> /bus_neg_salida
- J2 pad 14: unconnected-(J2-Pin_14-Pad14) -> /medicion_corriente
- J2 pad 23: unconnected-(J2-Pin_23-Pad23) -> /llave_de_emergencia
- Jsalida_1 pad 1: /Bit_1 -> /Vcc_out
- Jsalida_1 pad 10: GND -> /bus_pos_1
- Jsalida_1 pad 11: /clock -> /Bit_2
- Jsalida_1 pad 12: /latch -> /salida_adc_1
- Jsalida_1 pad 13: /Vcc_out -> /Bit_1
- Jsalida_1 pad 14: /Data_1 -> /Bit_0
- Jsalida_1 pad 2: /Bit_0 -> /Data_1
- Jsalida_1 pad 3: /Bit_2 -> /clock
- Jsalida_1 pad 4: /salida_adc_1 -> /latch
- Jsalida_1 pad 5: /bus_pos_1 -> GND
- Jsalida_1 pad 6: /bus_pos_1 -> GND
- Jsalida_1 pad 9: GND -> /bus_pos_1
- Jsalida_2 pad 1: /Bit_1 -> /Vcc_out
- Jsalida_2 pad 10: GND -> /bus_pos_2
- Jsalida_2 pad 11: /clock -> /Bit_2
- Jsalida_2 pad 12: /latch -> /salida_adc_2
- Jsalida_2 pad 13: /Vcc_out -> /Bit_1
- Jsalida_2 pad 14: /Data_2 -> /Bit_0
- Jsalida_2 pad 2: /Bit_0 -> /Data_2
- Jsalida_2 pad 3: /Bit_2 -> /clock
- Jsalida_2 pad 4: /salida_adc_2 -> /latch
- Jsalida_2 pad 5: /bus_pos_2 -> GND
- Jsalida_2 pad 6: /bus_pos_2 -> GND
- Jsalida_2 pad 9: GND -> /bus_pos_2
- Jsalida_3 pad 1: /Bit_1 -> /Vcc_out
- Jsalida_3 pad 10: GND -> /bus_pos_3
- Jsalida_3 pad 11: /clock -> /Bit_2
- Jsalida_3 pad 12: /latch -> /salida_adc_3
- Jsalida_3 pad 13: /Vcc_out -> /Bit_1
- Jsalida_3 pad 14: /Data_3 -> /Bit_0
- Jsalida_3 pad 2: /Bit_0 -> /Data_3
- Jsalida_3 pad 3: /Bit_2 -> /clock
- Jsalida_3 pad 4: /salida_adc_3 -> /latch
- Jsalida_3 pad 5: /bus_pos_3 -> GND
- Jsalida_3 pad 6: /bus_pos_3 -> GND
- Jsalida_3 pad 9: GND -> /bus_pos_3
- Jsalida_4 pad 1: /Bit_1 -> /Vcc_out
- Jsalida_4 pad 10: GND -> /bus_pos_4
- Jsalida_4 pad 11: /clock -> /Bit_2
- Jsalida_4 pad 12: /latch -> /salida_adc_4
- Jsalida_4 pad 13: /Vcc_out -> /Bit_1
- Jsalida_4 pad 14: /Data_4 -> /Bit_0
- Jsalida_4 pad 2: /Bit_0 -> /Data_4
- Jsalida_4 pad 3: /Bit_2 -> /clock
- Jsalida_4 pad 4: /salida_adc_4 -> /latch
- Jsalida_4 pad 5: /bus_pos_4 -> GND
- Jsalida_4 pad 6: /bus_pos_4 -> GND
- Jsalida_4 pad 9: GND -> /bus_pos_4
- SW1 pad 1: /Vcc -> Net-(Q2-D_1)
- SW1 pad 3: GND -> unconnected-(SW1-C-Pad3)
- SW2 pad 1: /bus_pos_1 -> /bus_pos_4
- SW2 pad 2: /bus_pos_2 -> /bus_pos_3
- SW2 pad 3: /bus_pos_3 -> /bus_pos_2
- SW2 pad 4: /bus_pos_4 -> /bus_pos_1
- TP1 pad 1: /bus_pos_salida -> /shunt
- TP2 pad 1: /bus_neg_1 -> /bus_neg_salida
- U3 pad 1: unconnected-(U3-Pad1) -> /medicion_corriente
- U3 pad 3: unconnected-(U3-+-Pad3) -> /bus_pos_salida
- U3 pad 4: unconnected-(U3---Pad4) -> /shunt
Routing:
- net /bus_neg_salida: track 0.00 -> 80.6 mm
- net /bus_pos_4: track 10.9 -> 78.8 mm
- net /bus_pos_1: track 20.1 -> 86.3 mm
- net Net-(U1B--): track 49.2 -> 0.00 mm
- net Net-(U1B-+): track 47.9 -> 0.00 mm
- net /bus_pos_2: track 28.6 -> 72.4 mm
- net Net-(U1C-+): track 34.7 -> 0.00 mm
- net Net-(U1C--): track 33.9 -> 0.00 mm
- net Net-(U1A-+): track 31.5 -> 0.00 mm
- net Net-(U1D-+): track 29.9 -> 0.00 mm
- net Net-(U1D--): track 27.7 -> 0.00 mm
- net /shunt: track 0.00 -> 23.9 mm
- net (no net): track 0.00 -> 21.6 mm
- net /Vcc_neg: track 20.5 -> 0.00 mm
- net /source: track 0.00 -> 17.4 mm
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
Commit message: conexiones de los integrados y sus resistencias
Parts:
- removed C4: 100n, Capacitor_SMD:C_1206_3216Metric_Pad1.33x1.80mm_HandSolder
- added C5: 100n, Capacitor_SMD:C_1206_3216Metric_Pad1.33x1.80mm_HandSolder, F.Cu at (431.4, 97.3)
- added C6: 100n, Capacitor_SMD:C_1206_3216Metric_Pad1.33x1.80mm_HandSolder, F.Cu at (418.5, 89.6)
- added C7: 100n, Capacitor_SMD:C_1206_3216Metric_Pad1.33x1.80mm_HandSolder, F.Cu at (456.7, 85.3)
- added C8: 100n, Capacitor_SMD:C_1206_3216Metric_Pad1.33x1.80mm_HandSolder, F.Cu at (448.1, 93.5)
- added J5: Conn_01x03_Pin, Connector_PinHeader_1.27mm:PinHeader_1x03_P1.27mm_Vertical, B.Cu at (405.4, 155.0)
- Bornera2: moved to B.Cu
- R1: value 22k -> 10k
- moved G*** 277.1 mm to (447.3, 137.7)
- moved Rf3 57.5 mm to (465.3, 90.2)
- moved Rx4 55.5 mm to (446.7, 85.3), turned to 180 degrees
- moved Rx3 54.3 mm to (463.8, 86.1)
- moved C3 52.2 mm to (431.1, 86.0), turned to -90 degrees
- moved Bornera2 50.4 mm to (398.0, 149.8), turned to -90 degrees
- moved R4 48.7 mm to (409.9, 134.8), turned to -90 degrees
- moved R5 47.4 mm to (405.5, 144.7), turned to 180 degrees
- moved Rf2 45.4 mm to (463.9, 97.3), turned to 90 degrees
- moved Rf4 41.4 mm to (448.8, 90.7), turned to 0 degrees
- moved C2 41.3 mm to (436.6, 91.2), turned to 90 degrees
- moved Rf1 36.0 mm to (451.1, 99.8), turned to 180 degrees
- moved R41 34.5 mm to (452.3, 85.3), turned to 180 degrees
- moved R12 33.1 mm to (445.0, 101.5)
- moved Rx2 32.1 mm to (457.3, 107.1), turned to -90 degrees
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Connections:
- C3 pad 1: /Vcc_neg -> GND
- C3 pad 2: GND -> /Vcc_neg
- J1 pad 15: unconnected-(J1-Pin_15-Pad15) -> /Vcc_stm
- J1 pad 17: /Vcc -> unconnected-(J1-Pin_17-Pad17)
Routing:
- net /Vcc_stm: track 0.00 -> 87.6 mm
- net /Vcc_out: track 25.6 -> 70.7 mm
- net (no net): track 21.6 -> 0.00 mm
- net Net-(U1A-+): track 0.00 -> 19.7 mm
- net Net-(U1D--): track 0.00 -> 19.0 mm
- net /gate: track 0.00 -> 18.2 mm
- net /bus_pos_3: track 60.2 -> 76.5 mm
- net Net-(U1C--): track 0.00 -> 16.1 mm
- net /bus_pos_2: track 72.4 -> 87.0 mm
- net Net-(U1C-+): track 0.00 -> 13.8 mm
- net /llave_de_emergencia: track 0.07 -> 13.0 mm
- net Net-(U1A--): track 0.00 -> 11.9 mm
- net Net-(U1B--): track 0.00 -> 11.4 mm
- net Net-(U1D-+): track 0.00 -> 11.0 mm
- net Net-(U1B-+): track 0.00 -> 10.2 mm
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Other:
- board outline added: 120 x 131.5 mm
