File: hardware/Circuito Final/Circuito externo/Circuito Final - Circuito externo.kicad_pcb (KiCad board)
At the start: 2 copper layers, 120 x 131.5 mm, 55 parts, among them J1 Conn_02x19_Odd_Even, J2 Conn_02x19_Odd_Even, J3 Conn_01x02, J4 Conn_01x02, J5 Conn_01x03_Pin, Q1 FDMS6681Z, Q2 FDMS6681Z, Q3 MMBT2222A, SW1 SW_SPDT, SW2 SW_DIP_x04, SW3 SW_DIP_x04, SW4 SW_DIP_x01, SW5 SW_DIP_x01, SW6 SW_DIP_x01, U1 Opamp_Quad, U2 ICL7660, U3 INA180A1

Commit message: conectores de banco ruteados
Parts:
- added R33: 0, Resistor_SMD:R_1206_3216Metric_Pad1.30x1.75mm_HandSolder, F.Cu at (441.4, 99.4)
- added R34: 0, Resistor_SMD:R_1206_3216Metric_Pad1.30x1.75mm_HandSolder, B.Cu at (473.8, 46.3)
- added R35: 0, Resistor_SMD:R_1206_3216Metric_Pad1.30x1.75mm_HandSolder, F.Cu at (483.9, 35.0)
- added R36: 0, Resistor_SMD:R_1206_3216Metric_Pad1.30x1.75mm_HandSolder, B.Cu at (406.4, 47.2)
- added R37: 0, Resistor_SMD:R_1206_3216Metric_Pad1.30x1.75mm_HandSolder, F.Cu at (392.7, 47.6)
- added R38: 0, Resistor_SMD:R_1206_3216Metric_Pad1.30x1.75mm_HandSolder, F.Cu at (465.2, 144.5)
- added R39: 0, Resistor_SMD:R_1206_3216Metric_Pad1.30x1.75mm_HandSolder, F.Cu at (395.8, 141.4)
- added R40: 0, Resistor_SMD:R_1206_3216Metric_Pad1.30x1.75mm_HandSolder, F.Cu at (397.2, 126.1)
- J5: footprint Connector_PinHeader_1.27mm:PinHeader_1x03_P1.27mm_Vertical -> Connector_PinHeader_2.54mm:PinHeader_1x03_P2.54mm_Vertical
- moved SW1 10.1 mm to (396.8, 116.9)
- moved R12 5.98 mm to (450.4, 104.1), turned to -90 degrees
- moved Rf2 3.66 mm to (462.7, 100.8), turned to 0 degrees
- moved TP1 3.48 mm to (400.9, 97.1)
- moved TP2 3.45 mm to (400.9, 81.3)
- moved C8 1.69 mm to (446.5, 93.3)
- moved R22 1.55 mm to (462.7, 103.9)
- moved R42 1.40 mm to (443.0, 96.1), turned to 180 degrees
- moved Rf4 1.23 mm to (448.7, 89.5), turned to -90 degrees
Connections:
- C8 pad 2: /Vcc_out -> Net-(U1E-V+)
- J2 pad 2: /Bit_0 -> /Bit_2
- J2 pad 3: /Bit_2 -> /Bit_0
- U1 pad 4: /Vcc_out -> Net-(U1E-V+)
Routing:
- net /latch: track 0.00 -> 227.5 mm, vias 0 -> 3
- net /Bit_0: track 0.00 -> 216.4 mm, vias 0 -> 3
- net /Bit_2: track 0.00 -> 184.5 mm, vias 0 -> 1
- net /clock: track 0.00 -> 182.8 mm, vias 0 -> 4
- net /Bit_1: track 0.00 -> 179.9 mm, vias 0 -> 1
- net /salida_adc_3: track 0.00 -> 151.5 mm
- net /salida_adc_2: track 0.00 -> 132.2 mm, vias 0 -> 1
- net /Data_2: track 0.00 -> 111.4 mm, vias 0 -> 2
- net /Data_3: track 0.00 -> 99.7 mm, vias 0 -> 3
- net /Data_4: track 0.00 -> 87.8 mm
- net /bus_pos_2: track 87.0 -> 170.1 mm, vias 0 -> 1
- net /bus_pos_1: track 90.8 -> 169.0 mm, vias 0 -> 1
- net /banco2_med: track 3.50 -> 75.4 mm
- net /Data_1: track 0.00 -> 71.8 mm
- net /salida_adc_4: track 0.00 -> 67.3 mm
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
Commit message: faltan las conexiones a gnd
Parts:
- added R43: 0, Resistor_SMD:R_1206_3216Metric_Pad1.30x1.75mm_HandSolder, F.Cu at (77.6, 62.3)
- added R44: 0, Resistor_SMD:R_1206_3216Metric_Pad1.30x1.75mm_HandSolder, F.Cu at (89.9, 111.1)
- added R45: 0, Resistor_SMD:R_1206_3216Metric_Pad1.30x1.75mm_HandSolder, F.Cu at (92.8, 97.9)
- moved C3 350.2 mm to (81.1, 97.8)
- moved R36 348.9 mm to (57.7, 58.9)
- moved C8 348.8 mm to (97.9, 105.0)
- moved G*** 348.3 mm to (99.2, 149.4)
- moved R4 347.7 mm to (62.4, 146.2)
- moved Jsalida_2 347.3 mm to (139.3, 53.6)
- moved R35 347.3 mm to (136.8, 46.7)
- moved C1 347.3 mm to (56.7, 100.7)
- moved C2 347.3 mm to (89.6, 102.8)
- moved C5 347.3 mm to (84.4, 109.0)
- moved J1 347.3 mm to (128.5, 119.2)
- moved J2 347.3 mm to (67.6, 119.2)
- moved J5 347.3 mm to (58.3, 166.6)
- moved Jsalida_1 347.3 mm to (149.1, 74.6)
- moved Jsalida_3 347.3 mm to (75.6, 53.6)
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Routing:
- net /Vcc_out: track 28.5 -> 202.3 mm, vias 0 -> 6
- net GND: track 10.5 -> 167.8 mm, vias 0 -> 2
- net /salida_adc_1: track 0.00 -> 144.1 mm, vias 0 -> 2
- net /banco4_med: track 4.66 -> 68.8 mm, vias 0 -> 2
- net /bus_neg_1: track 54.1 -> 115.0 mm
- net /banco1_med: track 6.65 -> 67.6 mm, vias 0 -> 2
- net /banco3_med: track 4.15 -> 56.3 mm, vias 0 -> 2
- net /medicion_corriente: track 0.00 -> 42.6 mm, vias 0 -> 2
- net /bus_pos_2: track 170.1 -> 162.1 mm
- net /Bit_2: track 184.5 -> 189.0 mm
- net /Bit_1: track 179.9 -> 183.6 mm
- net /Data_3: track 99.7 -> 102.6 mm
- net /gate: track 18.2 -> 20.6 mm
- net /bus_pos_salida: track 71.8 -> 69.4 mm
- net /bus_neg_salida: track 75.8 -> 78.2 mm
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
Commit message: ya esta todo conectado, spoiler: un quilombo
Parts:
- added R46: 0, Resistor_SMD:R_1206_3216Metric_Pad1.30x1.75mm_HandSolder, F.Cu at (121.5, 94.4)
- added R47: 0, Resistor_SMD:R_1206_3216Metric_Pad1.30x1.75mm_HandSolder, F.Cu at (121.7, 168.0)
- added R48: 0, Resistor_SMD:R_1206_3216Metric_Pad1.30x1.75mm_HandSolder, B.Cu at (58.6, 111.2)
Routing:
- net GND: track 167.8 -> 510.7 mm, vias 2 -> 7
- net /Vcc_out: track 202.3 -> 260.3 mm
- net /Vcc_neg: track 6.31 -> 47.1 mm, vias 0 -> 2
- net /bus_pos_salida: track 69.4 -> 75.1 mm
- net Net-(U1E-V+): track 21.5 -> 23.8 mm
- net /banco2_med: track 75.4 -> 77.5 mm
- net /bus_pos_2: track 162.1 -> 163.5 mm
- net /Data_3: track 102.6 -> 101.3 mm
- net /Vcc_stm: track 87.6 -> 88.8 mm
- added copper zone on B.Cu, net GND
- added copper zone on F.Cu, net GND
