File: hardware/PCB/prototipo.kicad_sch (KiCad schematic)
At the start: 18 parts, among them J1 Conn_02x12_Odd_Even

Commit message: agranda los pads de las vias a 1.7mm
Parts:
- A1: value ~ -> (none)
